Commit message: updated world file

File: src/wheelchair_description/urdf/wheelchair.xacro (robot description, xacro)
@@ -6,5 +6,5 @@
   <xacro:property name="legs_length" value="0.01" />
   <xacro:property name="legs_height" value="0.0354" />
-  <xacro:property name="legs_weight" value="2" />
+  <xacro:property name="legs_weight" value="1" />
   <xacro:property name="main_wheel_length" value="0.0356884" />
   <xacro:property name="main_wheel_radius" value="0.201784" />
@@ -16,5 +16,5 @@
   <xacro:property name="chair_length" value="${3/2*main_wheel_radius}" /> <!-- From front wheel joint to back wheel joint -->
   <xacro:property name="chair_height" value="0.01" /> <!-- From front wheel joint to head rest -->
-  <xacro:property name="chair_weight" value="50.0" />
+  <xacro:property name="chair_weight" value="70.0" />
   <xacro:include filename="$(find wheelchair_description)/urdf/wheelchair.gazebo" />
   <xacro:include filename="$(find wheelchair_description)/urdf/materials.xacro" />

File: wheelchair.urdf (robot description, URDF)
Before this commit: robot wheelchair, 13 links, 12 joints
Links:
- removed link left_leg_b
- removed link right_leg_b
- link base: mass 50.0 -> 70.0
- link l_rev: mass 0.1 -> 1
- link left_leg: mass 0.1 -> 1
- link r_rev: mass 0.1 -> 1
- link right_leg: mass 0.1 -> 1
Joints:
- removed joint l_rev_left_leg_b_joint
- removed joint left_leg_b_lf_joint
- removed joint r_rev_right_leg_b_joint
- removed joint right_leg_b_rf_joint
- added joint l_rev_lf_joint: type continuous, parent l_rev, child lf, origin xyz=0.04 0 -0.096 rpy=0 0 0, axis 0 1 0, limit effort=100 velocity=100
- added joint r_rev_rf_joint: type continuous, parent r_rev, child rf, origin xyz=0.04 0 -0.096 rpy=0 0 0, axis 0 1 0, limit effort=100 velocity=100
