Commit message: modified

File: src/wheelchair_description/urdf/macros.xacro (robot description, xacro)
@@ -26,5 +26,5 @@
       <axis xyz="${axis}" rpy="0 0 0"/>
       <limit effort="100" velocity="100"/>
-      <joint_properties damping="0.0" friction="0.0"/>
+      <joint_properties damping="0.1" friction="0.1"/>
     </joint>
   </xacro:macro>

File: src/wheelchair_description/urdf/wheelchair.urdf (robot description, URDF)
Before this commit: robot wheelchair, 13 links, 12 joints
Links:
- removed link left_leg_b
- removed link right_leg_b
- link l_rev: mass 0.1 -> 2
- link left_leg: mass 0.1 -> 2
- link r_rev: mass 0.1 -> 2
- link right_leg: mass 0.1 -> 2
Joints:
- removed joint l_rev_left_leg_b_joint
- removed joint left_leg_b_lf_joint
- removed joint r_rev_right_leg_b_joint
- removed joint right_leg_b_rf_joint
- added joint l_rev_lf_joint: type continuous, parent l_rev, child lf, origin xyz=0.04 0 -0.096 rpy=0 0 0, axis 0 1 0, limit effort=100 velocity=100
- added joint r_rev_rf_joint: type continuous, parent r_rev, child rf, origin xyz=0.04 0 -0.096 rpy=0 0 0, axis 0 1 0, limit effort=100 velocity=100

File: src/wheelchair_description/urdf/wheelchair.xacro (robot description, xacro)
@@ -6,5 +6,5 @@
   <xacro:property name="legs_length" value="0.01" />
   <xacro:property name="legs_height" value="0.0354" />
-  <xacro:property name="legs_weight" value="0.1" />
+  <xacro:property name="legs_weight" value="2" />
   <xacro:property name="main_wheel_length" value="0.0356884" />
   <xacro:property name="main_wheel_radius" value="0.201784" />
@@ -65,10 +65,14 @@
   <wheel  lr="l_rev" tY="0.02" xyz=" 0 0 0" rpy="0 0 0" wheelWidth="${main_wheel_length}" wheelRadius="${legs_width}" wheelMass="${legs_weight}" meshFile="wheelchair_wheel_rev"/>
   <wheel_joint parent="left_leg" child ="l_rev" xyz="0 0 ${-legs_height}" rpy="0 0 0" axis="0 0 1"/>
-  <chassis name="left_leg_b" xyz="0 0 ${-0.1065/2}" rpy="0 0 0" m="${legs_weight}" chassisLength="${legs_length}" chassisWidth="${legs_width}" chassisHeight="0.1065"/>
+ <!--
+  <chassis name="left_leg_b" xyz="0 0 ${-small_wheel_radius}" rpy="0 0 0" m="${legs_weight}" chassisLength="${legs_length}" chassisWidth="${legs_width}" chassisHeight="${2*small_wheel_radius}"/>
   <link_joint parent="l_rev" child ="left_leg_b" xyz="0 0 0" rpy="0 0 0" type="fixed"/>
+-->
   <wheel  lr="r_rev" tY="0.02" xyz=" 0 0 0" rpy="0 0 0" wheelWidth="${main_wheel_length}" wheelRadius="${legs_width}" wheelMass="${legs_weight}" meshFile="wheelchair_wheel_rev"/>
   <wheel_joint parent="right_leg" child ="r_rev" xyz="0 0 ${-legs_height}" rpy="0 0 0" axis="0 0 1"/>
-  <chassis name="right_leg_b" xyz="0 0 ${-0.1065/2}" rpy="0 0 0" m="${legs_weight}" chassisLength="${legs_length}" chassisWidth="${legs_width}" chassisHeight="0.1065"/>
+<!--
+  <chassis name="right_leg_b" xyz="0 0 ${-small_wheel_radius}" rpy="0 0 0" m="${legs_weight}" chassisLength="${legs_length}" chassisWidth="${legs_width}" chassisHeight="${2*small_wheel_radius}"/>
   <link_joint parent="r_rev" child ="right_leg_b" xyz="0 0 0" rpy="0 0 0" type="fixed"/>
+-->
   <wheel  lr="l" tY="0.02" xyz=" 0 0 0" rpy="${-pi/2} 0 0" wheelWidth="${main_wheel_length}" wheelRadius="${main_wheel_radius}" wheelMass="${main_wheel_weight}" meshFile="wheelchair_wheel"/>
   <wheel_joint parent="axel" child ="l" xyz="0 ${main_wheel_radius} 0" rpy="0 0 0" axis="0 1 0"/>
@@ -76,6 +80,6 @@
   <wheel_joint parent="axel" child ="r" xyz="0 ${-main_wheel_radius} 0" rpy="0 0 0" axis="0 1 0"/>
   <wheel  lr="lf" tY="0.001" xyz=" 0 0 0" rpy="${pi/2} 0 0" wheelWidth="${small_wheel_length}" wheelRadius="${small_wheel_radius}" wheelMass="${small_wheel_weight}" meshFile="wheelchair_wheel_small"/>
-  <wheel_joint parent="left_leg_b" child ="lf" xyz="0 0 ${-0.1065}" rpy="0 0 0" axis="0 1 0"/>
+  <wheel_joint parent="l_rev" child ="lf" xyz="0.04 0 ${-2*small_wheel_radius+0.04}" rpy="0 0 0" axis="0 1 0"/>
   <wheel  lr="rf" tY="0.001" xyz=" 0 0 0" rpy="${pi/2} 0 0" wheelWidth="${small_wheel_length}" wheelRadius="${small_wheel_radius}" wheelMass="${small_wheel_weight}" meshFile="wheelchair_wheel_small"/>
-  <wheel_joint parent="right_leg_b" child ="rf" xyz="0 0 ${-0.1065}" rpy="0 0 0" axis="0 1 0"/>
+  <wheel_joint parent="r_rev" child ="rf" xyz="0.04 0 ${-2*small_wheel_radius + 0.04}" rpy="0 0 0" axis="0 1 0"/>
 </robot>

Commit message: updated dimenstion and dynamics

File: src/wheelchair_description/urdf/macros.xacro (robot description, xacro)
@@ -26,5 +26,5 @@
       <axis xyz="${axis}" rpy="0 0 0"/>
       <limit effort="100" velocity="100"/>
-      <joint_properties damping="0.1" friction="0.1"/>
+      <joint_properties damping="0.01" friction="0.5"/>
     </joint>
   </xacro:macro>

File: src/wheelchair_description/urdf/wheelchair.xacro (robot description, xacro)
@@ -1,10 +1,8 @@
 <?xml version='1.0'?>
 <robot name="wheelchair" xmlns:xacro="http://www.ros.org/wiki/xacro" >
-  <xacro:property name="cameraSize" value="0.05"/>
-  <xacro:property name="cameraMass" value="0.1"/>
   <xacro:property name="legs_width" value="0.01" />
   <xacro:property name="legs_length" value="0.01" />
   <xacro:property name="legs_height" value="0.0354" />
-  <xacro:property name="legs_weight" value="1" />
+  <xacro:property name="legs_weight" value="0.25" />
   <xacro:property name="main_wheel_length" value="0.0356884" />
   <xacro:property name="main_wheel_radius" value="0.201784" />
@@ -12,9 +10,13 @@
   <xacro:property name="small_wheel_radius" value="0.068" />
   <xacro:property name="small_wheel_length" value="0.032" />
-  <xacro:property name="small_wheel_weight" value="1.0" />
+  <xacro:property name="small_wheel_weight" value="1.5" />
   <xacro:property name="chair_width" value="${2*main_wheel_radius - 0.2}" /> <!-- From front wheel right joint to front wheel left joint -->
-  <xacro:property name="chair_length" value="${3/2*main_wheel_radius}" /> <!-- From front wheel joint to back wheel joint -->
-  <xacro:property name="chair_height" value="0.01" /> <!-- From front wheel joint to head rest -->
-  <xacro:property name="chair_weight" value="70.0" />
+  <xacro:property name="chair_length" value="${3/2*main_wheel_radius}" /> 	 <!-- From front wheel joint to back wheel joint -->
+  <xacro:property name="chair_height" value="0.01" /> 						 <!-- From front wheel joint to head rest -->
+  <xacro:property name="chair_weight" value="3.0" />
+  <xacro:property name="axle_width" value="0.01" />
+  <xacro:property name="axle_length" value="${2*main_wheel_radius}"/>
+  <xacro:property name="axle_height" value="0.01" />
+  <xacro:property name="axle_weight" value="2.0" />
   <xacro:include filename="$(find wheelchair_description)/urdf/wheelchair.gazebo" />
   <xacro:include filename="$(find wheelchair_description)/urdf/materials.xacro" />
@@ -34,14 +36,14 @@
   </visual>
   </link>
-  <link name='axel'>
+  <link name='axle'>
     <inertial>
       <origin xyz="0 0 0" rpy=" 0 0 0"/>
-      <mass value="50.0"/>
-      <box_inertia m="50" x="0.01" y="0.406054" z ="0.01" />
+      <mass value="${axle_weight}"/>
+      <box_inertia m="${axle_weight}" x="${axle_width}" y="${axle_length}" z ="${axle_height}" />
     </inertial>
     <collision name='collision'>
-      <origin xyz="0 0 0}" rpy=" 0 0 0"/>
+      <origin xyz="0 0 0" rpy=" 0 0 0"/>
       <geometry>
-        <box size="0.01 0.406054 0.01"/>
+        <box size="${axle_width} ${axle_length} ${axle_height}"/>
       </geometry>
     </collision>
@@ -49,37 +51,26 @@
       <origin xyz="0 0 0" rpy=" 0 0 0"/>
       <geometry>
-        <box size="0.01 0.406054 0.01"/>
+        <box size="${axle_width} ${axle_length} ${axle_height}"/>
       </geometry>
     </visual>
   </link>
-  <!--
-  <chassis name="base" xyz="0 0 ${main_wheel_radius}" rpy="0 0 0" m="2" chassisLength="0.01" chassisWidth="${2*main_wheel_radius}" chassisHeight="0.01"/>
--->
-  <link_joint parent="footprint" child ="axel" xyz="0 0 ${main_wheel_radius}" rpy="0 0 0" type="fixed"/>
+  <link_joint parent="footprint" child ="axle" xyz="0 0 ${main_wheel_radius}" rpy="0 0 0" type="fixed"/>
   <chassis name="base" xyz="${chair_length/2} 0 0" rpy="0 0 0" m="${chair_weight}" chassisLength="${chair_length}" chassisWidth="${chair_width}" chassisHeight="${chair_height}"/>
-  <link_joint parent="axel" child ="base" xyz="0 0 0" rpy="0 0 0" type="fixed"/>
-  <chassis name="left_leg" xyz="0 0 ${-legs_height/2}" rpy="0 0 0" m="${legs_weight}" chassisLength="${legs_length}" chassisWidth="${legs_width}" chassisHeight="${legs_height}"/>
-  <link_joint parent="base" child ="left_leg" xyz="${chair_length} ${chair_width/2} 0" rpy="0 0 0" type="fixed"/>
-  <chassis name="right_leg" xyz="0 0 ${-legs_height/2}" rpy="0 0 0" m="${legs_weight}" chassisLength="${legs_length}" chassisWidth="${legs_width}" chassisHeight="${legs_height}"/>
-  <link_joint parent="base" child ="right_leg" xyz="${chair_length} ${-chair_width/2} 0" rpy="0 0 0" type="fixed"/>
-  <wheel  lr="l_rev" tY="0.02" xyz=" 0 0 0" rpy="0 0 0" wheelWidth="${main_wheel_length}" wheelRadius="${legs_width}" wheelMass="${legs_weight}" meshFile="wheelchair_wheel_rev"/>
-  <wheel_joint parent="left_leg" child ="l_rev" xyz="0 0 ${-legs_height}" rpy="0 0 0" axis="0 0 1"/>
- <!--
-  <chassis name="left_leg_b" xyz="0 0 ${-small_wheel_radius}" rpy="0 0 0" m="${legs_weight}" chassisLength="${legs_length}" chassisWidth="${legs_width}" chassisHeight="${2*small_wheel_radius}"/>
-  <link_joint parent="l_rev" child ="left_leg_b" xyz="0 0 0" rpy="0 0 0" type="fixed"/>
--->
-  <wheel  lr="r_rev" tY="0.02" xyz=" 0 0 0" rpy="0 0 0" wheelWidth="${main_wheel_length}" wheelRadius="${legs_width}" wheelMass="${legs_weight}" meshFile="wheelchair_wheel_rev"/>
-  <wheel_joint parent="right_leg" child ="r_rev" xyz="0 0 ${-legs_height}" rpy="0 0 0" axis="0 0 1"/>
-<!--
-  <chassis name="right_leg_b" xyz="0 0 ${-small_wheel_radius}" rpy="0 0 0" m="${legs_weight}" chassisLength="${legs_length}" chassisWidth="${legs_width}" chassisHeight="${2*small_wheel_radius}"/>
-  <link_joint parent="r_rev" child ="right_leg_b" xyz="0 0 0" rpy="0 0 0" type="fixed"/>
--->
-  <wheel  lr="l" tY="0.02" xyz=" 0 0 0" rpy="${-pi/2} 0 0" wheelWidth="${main_wheel_length}" wheelRadius="${main_wheel_radius}" wheelMass="${main_wheel_weight}" meshFile="wheelchair_wheel"/>
-  <wheel_joint parent="axel" child ="l" xyz="0 ${main_wheel_radius} 0" rpy="0 0 0" axis="0 1 0"/>
-  <wheel  lr="r" tY="0.02" xyz=" 0 0 0" rpy="${pi/2} 0 0" wheelWidth="${main_wheel_length}" wheelRadius="${main_wheel_radius}" wheelMass="${main_wheel_weight}" meshFile="wheelchair_wheel"/>
-  <wheel_joint parent="axel" child ="r" xyz="0 ${-main_wheel_radius} 0" rpy="0 0 0" axis="0 1 0"/>
-  <wheel  lr="lf" tY="0.001" xyz=" 0 0 0" rpy="${pi/2} 0 0" wheelWidth="${small_wheel_length}" wheelRadius="${small_wheel_radius}" wheelMass="${small_wheel_weight}" meshFile="wheelchair_wheel_small"/>
-  <wheel_joint parent="l_rev" child ="lf" xyz="0.04 0 ${-2*small_wheel_radius+0.04}" rpy="0 0 0" axis="0 1 0"/>
-  <wheel  lr="rf" tY="0.001" xyz=" 0 0 0" rpy="${pi/2} 0 0" wheelWidth="${small_wheel_length}" wheelRadius="${small_wheel_radius}" wheelMass="${small_wheel_weight}" meshFile="wheelchair_wheel_small"/>
-  <wheel_joint parent="r_rev" child ="rf" xyz="0.04 0 ${-2*small_wheel_radius + 0.04}" rpy="0 0 0" axis="0 1 0"/>
+  <link_joint parent="axle" child ="base" xyz="0 0 0" rpy="0 0 0" type="fixed"/>
+  <chassis name="front_left_leg" xyz="0 0 ${-legs_height/2}" rpy="0 0 0" m="${legs_weight}" chassisLength="${legs_length}" chassisWidth="${legs_width}" chassisHeight="${legs_height}"/>
+  <link_joint parent="base" child ="front_left_leg" xyz="${chair_length} ${chair_width/2} 0" rpy="0 0 0" type="fixed"/>
+  <chassis name="front_right_leg" xyz="0 0 ${-legs_height/2}" rpy="0 0 0" m="${legs_weight}" chassisLength="${legs_length}" chassisWidth="${legs_width}" chassisHeight="${legs_height}"/>
+  <link_joint parent="base" child ="front_right_leg" xyz="${chair_length} ${-chair_width/2} 0" rpy="0 0 0" type="fixed"/>
+  <wheel  lr="front_left_leg_rev" tY="0.02" xyz=" 0 0 0" rpy="0 0 0" wheelWidth="${main_wheel_length}" wheelRadius="${legs_width}" wheelMass="${legs_weight}" meshFile="wheelchair_wheel_rev"/>
+  <wheel_joint parent="front_left_leg" child ="front_left_leg_rev" xyz="0 0 ${-legs_height}" rpy="0 0 0" axis="0 0 1"/>
+  <wheel  lr="front_right_rev" tY="0.02" xyz=" 0 0 0" rpy="0 0 0" wheelWidth="${main_wheel_length}" wheelRadius="${legs_width}" wheelMass="${legs_weight}" meshFile="wheelchair_wheel_rev"/>
+  <wheel_joint parent="front_right_leg" child ="front_right_rev" xyz="0 0 ${-legs_height}" rpy="0 0 0" axis="0 0 1"/>
+  <wheel  lr="rear_left_wheel" tY="0.02" xyz=" 0 0 0" rpy="${-pi/2} 0 0" wheelWidth="${main_wheel_length}" wheelRadius="${main_wheel_radius}" wheelMass="${main_wheel_weight}" meshFile="wheelchair_wheel"/>
+  <wheel_joint parent="axle" child ="rear_left_wheel" xyz="0 ${main_wheel_radius} 0" rpy="0 0 0" axis="0 1 0"/>
+  <wheel  lr="rear_right_wheel" tY="0.02" xyz=" 0 0 0" rpy="${pi/2} 0 0" wheelWidth="${main_wheel_length}" wheelRadius="${main_wheel_radius}" wheelMass="${main_wheel_weight}" meshFile="wheelchair_wheel"/>
+  <wheel_joint parent="axle" child ="rear_right_wheel" xyz="0 ${-main_wheel_radius} 0" rpy="0 0 0" axis="0 1 0"/>
+  <wheel  lr="front_left_wheel" tY="0.001" xyz=" 0 0 0" rpy="${pi/2} 0 0" wheelWidth="${small_wheel_length}" wheelRadius="${small_wheel_radius}" wheelMass="${small_wheel_weight}" meshFile="wheelchair_wheel_small"/>
+  <wheel_joint parent="l_front_left_leg_rev" child ="front_left_wheel" xyz="0.04 0 ${-2*small_wheel_radius+0.04}" rpy="0 0 0" axis="0 1 0"/>
+  <wheel  lr="front_right_wheel" tY="0.001" xyz=" 0 0 0" rpy="${pi/2} 0 0" wheelWidth="${small_wheel_length}" wheelRadius="${small_wheel_radius}" wheelMass="${small_wheel_weight}" meshFile="wheelchair_wheel_small"/>
+  <wheel_joint parent="front_right_rev" child ="front_right_wheel" xyz="0.04 0 ${-2*small_wheel_radius + 0.04}" rpy="0 0 0" axis="0 1 0"/>
 </robot>
