Commit message: added simulation

File: src/wheelchair_description/urdf/wheelchair.urdf (robot description, URDF)
Before this commit: robot wheelchair, 11 links, 10 joints
Links:
- removed link axel
- removed link l
- removed link l_rev
- removed link left_leg
- removed link lf
- removed link r
- removed link r_rev
- removed link rf
- removed link right_leg
- added link axle, mass 2.0; collision box size=0.01 0.403568 0.01; visual box size=0.01 0.403568 0.01
- added link front_left_leg, mass 0.25; collision box size=0.01 0.01 0.0354; visual box size=0.01 0.01 0.0354
- added link front_left_leg_rev, mass 0.25; collision cylinder length=0.0356884 radius=0.01; visual mesh filename=package://wheelchair_description/meshes/wheelchair_wheel_re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 scale=0.01 0.01 0.01
- added link front_left_wheel, mass 1.5; collision cylinder length=0.032 radius=0.068; visual mesh filename=package://wheelchair_description/meshes/wheelchair_wheel_sm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 scale=0.01 0.01 0.01
- added link front_right_leg, mass 0.25; collision box size=0.01 0.01 0.0354; visual box size=0.01 0.01 0.0354
- added link front_right_leg_rev, mass 0.25; collision cylinder length=0.0356884 radius=0.01; visual mesh filename=package://wheelchair_description/meshes/wheelchair_wheel_re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 scale=0.01 0.01 0.01
- added link front_right_wheel, mass 1.5; collision cylinder length=0.032 radius=0.068; visual mesh filename=package://wheelchair_description/meshes/wheelchair_wheel_sm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 scale=0.01 0.01 0.01
- added link rl_wheel, mass 3.0; collision cylinder length=0.0356884 radius=0.201784; visual mesh filename=package://wheelchair_description/meshes/wheelchair_wheel.stl scale=0.01 0.01 0.01
- added link rr_wheel, mass 3.0; collision cylinder length=0.0356884 radius=0.201784; visual mesh filename=package://wheelchair_description/meshes/wheelchair_wheel.stl scale=0.01 0.01 0.01
- link base: mass 50.0 -> 3.0; geometry collision box size=0.250676 0.223568 0.01; visual box size=0.250676 0.223568 0.01
Joints:
- removed joint axel_base_joint
- removed joint axel_l_joint
- removed joint axel_r_joint
- removed joint base_left_leg_joint
- removed joint base_right_leg_joint
- removed joint footprint_axel_joint
- removed joint l_rev_lf_joint
- removed joint left_leg_l_rev_joint
- removed joint r_rev_rf_joint
- removed joint right_leg_r_rev_joint
- added joint axle_base_joint: type fixed, parent axle, child base, origin xyz=0 0 0 rpy=0 0 0
- added joint axle_rl_wheel_joint: type continuous, parent axle, child rl_wheel, origin xyz=0 0.201784 0 rpy=0 0 0, axis 0 1 0, limit effort=100 velocity=100
- added joint axle_rr_wheel_joint: type continuous, parent axle, child rr_wheel, origin xyz=0 -0.201784 0 rpy=0 0 0, axis 0 1 0, limit effort=100 velocity=100
- added joint base_front_left_leg_joint: type fixed, parent base, child front_left_leg, origin xyz=0.250676 0.111784 0 rpy=0 0 0
- added joint base_front_right_leg_joint: type fixed, parent base, child front_right_leg, origin xyz=0.250676 -0.111784 0 rpy=0 0 0
- added joint footprint_axle_joint: type fixed, parent footprint, child axle, origin xyz=0 0 0.201784 rpy=0 0 0
- added joint front_left_leg_front_left_leg_rev_joint: type continuous, parent front_left_leg, child front_left_leg_rev, origin xyz=0 0 -0.0354 rpy=0 0 0, axis 0 0 1, limit effort=100 velocity=100
- added joint front_left_leg_rev_front_left_wheel_joint: type continuous, parent front_left_leg_rev, child front_left_wheel, origin xyz=0.04 0 -0.096 rpy=0 0 0, axis 0 1 0, limit effort=100 velocity=100
- added joint front_right_leg_front_right_leg_rev_joint: type continuous, parent front_right_leg, child front_right_leg_rev, origin xyz=0 0 -0.0354 rpy=0 0 0, axis 0 0 1, limit effort=100 velocity=100
- added joint front_right_leg_rev_front_right_wheel_joint: type continuous, parent front_right_leg_rev, child front_right_wheel, origin xyz=0.04 0 -0.096 rpy=0 0 0, axis 0 1 0, limit effort=100 velocity=100

File: src/wheelchair_description/urdf/wheelchair.xacro (robot description, xacro)
@@ -11,6 +11,6 @@
   <xacro:property name="small_wheel_length" value="0.032" />
   <xacro:property name="small_wheel_weight" value="1.5" />
-  <xacro:property name="chair_width" value="${2*main_wheel_radius - 0.2}" /> <!-- From front wheel right joint to front wheel left joint -->
-  <xacro:property name="chair_length" value="${3/2*main_wheel_radius}" /> 	 <!-- From front wheel joint to back wheel joint -->
+  <xacro:property name="chair_width" value="${2*main_wheel_radius - 0.18}" /> <!-- From front wheel right joint to front wheel left joint -->
+  <xacro:property name="chair_length" value="${3/2*main_wheel_radius - 0.052}" /> 	 <!-- From front wheel joint to back wheel joint -->
   <xacro:property name="chair_height" value="0.01" /> 						 <!-- From front wheel joint to head rest -->
   <xacro:property name="chair_weight" value="3.0" />
