Commit message: merged

File: mdu.urdf (robot description, URDF)
Before this commit: robot mdu, 4 links, 3 joints
Links:
- removed link chassis
- added link axle, mass 2.0; collision box size=0.01 0.28 0.01; visual box size=0.01 0.28 0.01
- added link base, mass 10.0; collision box size=0.13 0.23 0.15; visual box size=0.13 0.23 0.15
- added link caster; collision sphere radius=0.0635; visual sphere radius=0.0635
- link footprint: geometry visual box size=0.01 0.01 0.01
- link rear_left_wheel: mass 2.0 -> 3.0
- link rear_right_wheel: mass 2.0 -> 3.0
Joints:
- removed joint chassis_rear_left_wheel_joint
- removed joint chassis_rear_right_wheel_joint
- removed joint footprint_chassis_joint
- added joint axle_base_joint: type fixed, parent axle, child base, origin xyz=0 0 0 rpy=0 0 0
- added joint axle_rear_left_wheel_joint: type continuous, parent axle, child rear_left_wheel, origin xyz=0 0.14 0 rpy=0 0 0, axis 0 1 0, limit effort=100 velocity=100
- added joint axle_rear_right_wheel_joint: type continuous, parent axle, child rear_right_wheel, origin xyz=0 -0.14 0 rpy=0 0 0, axis 0 1 0, limit effort=100 velocity=100
- added joint base_caster_joint: type fixed, parent base, child caster, origin xyz=0.0665 0 -0.0635 rpy=0 0 0
- added joint footprint_axle_joint: type fixed, parent footprint, child axle, origin xyz=0 0 0.127 rpy=0 0 0

File: src/mdu_description/urdf/mdu.xacro (robot description, xacro)
@@ -3,78 +3,62 @@
   <xacro:property name="main_wheel_length" value="0.05" />
   <xacro:property name="main_wheel_radius" value="0.127" />
-  <xacro:property name="main_wheel_weight" value="3.0" />
+  <xacro:property name="main_wheel_weight" value="2.0" />
   <xacro:property name="axle_width" value="0.01" />
   <xacro:property name="axle_length" value="${0.28}"/>
   <xacro:property name="axle_height" value="0.01" />
   <xacro:property name="axle_weight" value="2.0" />
-  <xacro:property name="chair_width" value="${axle_length  - 0.05}" /> <!-- From front wheel right joint to front wheel left joint -->
-  <xacro:property name="chair_length" value="${chair_width - 0.1}" /> 	 <!-- From front wheel joint to back wheel joint -->
-  <xacro:property name="chair_height" value="0.15" /> 				 <!-- From front wheel joint to head rest -->
-  <xacro:property name="chair_weight" value="${10.0}" />
+  <xacro:property name="chassis_width" value="${axle_length  - 0.05}" /> <!-- From front wheel right joint to front wheel left joint -->
+  <xacro:property name="chassis_length" value="${chassis_width + 0.1}" /> 	 <!-- From front wheel joint to back wheel joint -->
+  <xacro:property name="chassis_height" value="0.1" /> 				 <!-- From front wheel joint to head rest -->
+  <xacro:property name="chassis_weight" value="${6.0}" />
   <xacro:include filename="$(find mdu_description)/urdf/mdu.gazebo" />
   <xacro:include filename="$(find mdu_description)/urdf/materials.xacro" />
   <xacro:include filename="$(find mdu_description)/urdf/macros.xacro" />
-  <link name='footprint'>
-    <pose xyz="0 0 0" rpy=" 0 0 0"/>
-    <visual>
-      <origin xyz="0 0 0" rpy=" 0 0 0"/>
-    </visual>
-    <!--visual>
-      <origin xyz="0 0 0" rpy="0 0 -3.14"/>
+  <link name='chassis'>
+    <inertial name="chassis_intertial">
+        <origin xyz="0 0 0" rpy="0 0 0" />
+        <mass value="${chassis_weight}"/>
+        <box_inertia m="${chassis_weight}" x="${chassis_length}" y="${chassis_width}" z ="${chassis_height}" />
+      </inertial>
+    <collision name='collision'>
       <geometry>
-         <mesh filename="package://wheelchair_description/meshes/wheelchair_chasis.stl" scale="0.01 0.01 0.01"/>
-      </geometry>
-  </visual-->
-  </link>
-  <link name='axle'>
-    <inertial>
-      <origin xyz="0 0 0" rpy=" 0 0 0"/>
-      <mass value="${axle_weight}"/>
-      <box_inertia m="${axle_weight}" x="${axle_width}" y="${axle_length}" z ="${axle_height}" />
-    </inertial>
-    <collision name='collision'>
-      <origin xyz="0 0 0" rpy=" 0 0 0"/>
-      <geometry>
-        <box size="${axle_width} ${axle_length} ${axle_height}"/>
+        <box size="${chassis_length} ${chassis_width} ${chassis_height}"/>
       </geometry>
     </collision>
-    <visual>
-      <origin xyz="0 0 0" rpy=" 0 0 0"/>
+    <visual name='chassis_visual'>
+      <origin xyz="0 0 0" rpy="0 0 0" />
       <geometry>
-        <box size="${axle_width} ${axle_length} ${axle_height}"/>
+        <box size="${chassis_length} ${chassis_width} ${chassis_height}"/>
+      </geometry>
+    </visual>
+    <collision name='caster_collision'>
+      <origin xyz="${-(chassis_length/2 - (main_wheel_radius/2))} 0 ${-main_wheel_radius/2}" rpy=" 0 0 0"/>
+      <geometry>
+        <sphere radius="${(main_wheel_radius/2)}"/>
+      </geometry>
+      <surface>
+        <friction>
+          <ode>
+            <mu>0</mu>
+            <mu2>0</mu2>
+            <slip1>1.0</slip1>
+            <slip2>1.0</slip2>
+          </ode>
+        </friction>
+      </surface>
+    </collision>
+    <visual name='caster_visual'>
+      <origin xyz="${-(chassis_length/2 - (main_wheel_radius/2))} 0 ${-main_wheel_radius/2}" rpy=" 0 0 0"/>
+      <geometry>
+        <sphere radius="${(main_wheel_radius/2)}"/>
       </geometry>
     </visual>
   </link>
-  <link name='caster'>
-      <collision name='caster_collision'>
-	      <origin xyz="0 0 0" rpy=" 0 0 0"/>
-	      <geometry>
-		<sphere radius="${main_wheel_radius/2}"/>
-	      </geometry>
-	      <surface>
-		<friction>
-		  <ode>
-		    <mu>0</mu>
-		    <mu2>0</mu2>
-		    <slip1>1.0</slip1>
-		    <slip2>1.0</slip2>
-		  </ode>
-		</friction>
-	      </surface>
-    </collision>
-    <visual name='caster_visual'>
-      <origin xyz="0 0 0" rpy=" 0 0 0"/>
-      <geometry>
-        <sphere radius="${main_wheel_radius/2}"/>
-      </geometry>
-   </visual>
- </link>
-  <link_joint parent="footprint" child ="axle" xyz="0 0 ${main_wheel_radius}" rpy="0 0 0" type="fixed"/>
-  <chassis name="base" xyz="${chair_length/2} 0 0" rpy="0 0 0" m="${chair_weight}" chassisLength="${chair_length}" chassisWidth="${chair_width}" chassisHeight="${chair_height}"/>
-  <link_joint parent="axle" child ="base" xyz="0 0 0" rpy="0 0 0" type="fixed"/>
-  <link_joint parent="base" child ="caster" xyz="${chair_length -main_wheel_radius/2} 0 ${-main_wheel_radius/2}" rpy="0 0 0" type="fixed"/>
+  <link name='footprint'>
+  </link>
+  <link_joint parent='footprint' child='chassis' xyz="0 0 ${main_wheel_radius}" rpy="0 0 0" type="fixed"/>
   <wheel  lr="rear_left_wheel" tY="0.02" xyz=" 0 0 0" rpy="${-pi/2} 0 0" wheelWidth="${main_wheel_length}" wheelRadius="${main_wheel_radius}" wheelMass="${main_wheel_weight}" meshFile="wheelchair_wheel"/>
-  <wheel_joint parent="axle" child ="rear_left_wheel" xyz="0 ${axle_length/2} 0" rpy="0 0 0" axis="0 1 0"/>
+  <wheel_joint parent="chassis" child ="rear_left_wheel" xyz="0.04 ${chassis_width/2 +0.02} 0" rpy="0 0 0" axis="0 1 0"/>
   <wheel  lr="rear_right_wheel" tY="0.02" xyz=" 0 0 0" rpy="${pi/2} 0 0" wheelWidth="${main_wheel_length}" wheelRadius="${main_wheel_radius}" wheelMass="${main_wheel_weight}" meshFile="wheelchair_wheel"/>
-  <wheel_joint parent="axle" child ="rear_right_wheel" xyz="0 ${-axle_length/2} 0" rpy="0 0 0" axis="0 1 0"/>
+  <wheel_joint parent="chassis" child ="rear_right_wheel" xyz="0.04 ${-chassis_width/2 - 0.02} 0" rpy="0 0 0" axis="0 1 0"/>
 </robot>

File: src/wheelchair_description/urdf/wheelchair (copy).xacro (robot description, xacro)
@@ -3,5 +3,5 @@
   <xacro:property name="legs_width" value="0.01" />
   <xacro:property name="legs_length" value="0.01" />
-  <xacro:property name="legs_height" value="0.16" />
+  <xacro:property name="legs_height" value="0.0354" />
   <xacro:property name="legs_weight" value="0.25" />
   <xacro:property name="main_wheel_length" value="0.0356884" />
@@ -11,5 +11,5 @@
   <xacro:property name="small_wheel_length" value="0.032" />
   <xacro:property name="small_wheel_weight" value="1.5" />
-  <xacro:property name="chair_width" value="${2*main_wheel_radius - 0.08}" /> <!-- From front wheel right joint to front wheel left joint -->
+  <xacro:property name="chair_width" value="${2*main_wheel_radius - 0.18}" /> <!-- From front wheel right joint to front wheel left joint -->
   <xacro:property name="chair_length" value="${3/2*main_wheel_radius - 0.052}" /> 	 <!-- From front wheel joint to back wheel joint -->
   <xacro:property name="chair_height" value="0.01" /> 						 <!-- From front wheel joint to head rest -->
@@ -58,16 +58,16 @@
   <link_joint parent="footprint" child ="axle" xyz="0 0 ${main_wheel_radius}" rpy="0 0 0" type="fixed"/>
   <chassis name="base" xyz="${chair_length/2} 0 0" rpy="0 0 0" m="${chair_weight}" chassisLength="${chair_length}" chassisWidth="${chair_width}" chassisHeight="${chair_height}"/>
-  <link_joint parent="axle" child ="base" xyz="0 0 0.1" rpy="0 0 0" type="fixed"/>
+  <link_joint parent="axle" child ="base" xyz="0 0 0" rpy="0 0 0" type="fixed"/>
   <chassis name="front_left_leg" xyz="0 0 ${-legs_height/2}" rpy="0 0 0" m="${legs_weight}" chassisLength="${legs_length}" chassisWidth="${legs_width}" chassisHeight="${legs_height}"/>
   <link_joint parent="base" child ="front_left_leg" xyz="${chair_length} ${chair_width/2} 0" rpy="0 0 0" type="fixed"/>
    <chassis name="rear_left_leg" xyz="0 0 ${-(legs_height + 0.1)/2}" rpy="0 0 0" m="${legs_weight}" chassisLength="${legs_length}" chassisWidth="${legs_width}" chassisHeight="${legs_height + 0.1}"/>
-  <link_joint parent="base" child ="rear_left_leg" xyz="0 ${chair_width/2} 0" rpy="0 0 0" type="fixed"/>
+  <link_joint parent="base" child ="rear_left_leg" xyz="0 ${chair_width/2 + 0.05} 0" rpy="0 0 0" type="fixed"/>
 <chassis name="rear_right_leg" xyz="0 0 ${-(legs_height + 0.1)/2}" rpy="0 0 0" m="${legs_weight}" chassisLength="${legs_length}" chassisWidth="${legs_width}" chassisHeight="${legs_height +0.1}"/>
-  <link_joint parent="base" child ="rear_right_leg" xyz="0 ${-chair_width/2} 0" rpy="0 0 0" type="fixed"/>
+  <link_joint parent="base" child ="rear_right_leg" xyz="0 ${-chair_width/2 - 0.05} 0" rpy="0 0 0" type="fixed"/>
   <chassis name="front_right_leg" xyz="0 0 ${-legs_height/2}" rpy="0 0 0" m="${legs_weight}" chassisLength="${legs_length}" chassisWidth="${legs_width}" chassisHeight="${legs_height}"/>
   <link_joint parent="base" child ="front_right_leg" xyz="${chair_length} ${-chair_width/2} 0" rpy="0 0 0" type="fixed"/>
-  <wheel  lr="front_left_leg_rev" tY="0.02" xyz=" 0 0 0" rpy="0 0 0" wheelWidth="${0.1}" wheelRadius="${legs_width}" wheelMass="${legs_weight}" meshFile="wheelchair_wheel_rev"/>
+  <wheel  lr="front_left_leg_rev" tY="0.02" xyz=" 0 0 0" rpy="0 0 0" wheelWidth="${0.01}" wheelRadius="${legs_width}" wheelMass="${legs_weight}" meshFile="wheelchair_wheel_rev"/>
   <wheel_joint parent="front_left_leg" child ="front_left_leg_rev" xyz="0 0 ${-legs_height}" rpy="0 0 0" axis="0 0 1"/>
-  <wheel  lr="front_right_leg_rev" tY="0.02" xyz=" 0 0 0" rpy="0 0 0" wheelWidth="${0.1}" wheelRadius="${legs_width}" wheelMass="${legs_weight}" meshFile="wheelchair_wheel_rev"/>
+  <wheel  lr="front_right_leg_rev" tY="0.02" xyz=" 0 0 0" rpy="0 0 0" wheelWidth="${0.01}" wheelRadius="${legs_width}" wheelMass="${legs_weight}" meshFile="wheelchair_wheel_rev"/>
   <wheel_joint parent="front_right_leg" child ="front_right_leg_rev" xyz="0 0 ${-legs_height}" rpy="0 0 0" axis="0 0 1"/>
   <wheel  lr="rear_left_wheel" tY="0.02" xyz=" 0 0 0" rpy="${-pi/2} 0 0" wheelWidth="${main_wheel_length}" wheelRadius="${main_wheel_radius}" wheelMass="${main_wheel_weight}" meshFile="wheelchair_wheel"/>
@@ -76,6 +76,6 @@
   <wheel_joint parent="axle" child ="rear_right_wheel" xyz="0 ${-main_wheel_radius} 0" rpy="0 0 0" axis="0 1 0"/>
   <wheel  lr="front_left_wheel" tY="0.001" xyz=" 0 0 0" rpy="${pi/2} 0 0" wheelWidth="${small_wheel_length}" wheelRadius="${small_wheel_radius}" wheelMass="${small_wheel_weight}" meshFile="wheelchair_wheel_small"/>
-  <wheel_joint parent="front_left_leg_rev" child ="front_left_wheel" xyz="0.017 0 ${-0.07352}" rpy="0 0 0" axis="0 1 0"/>
+  <wheel_joint parent="front_left_leg_rev" child ="front_left_wheel" xyz="0.017 0 ${-2*small_wheel_radius+0.0377}" rpy="0 0 0" axis="0 1 0"/>
   <wheel  lr="front_right_wheel" tY="0.001" xyz=" 0 0 0" rpy="${pi/2} 0 0" wheelWidth="${small_wheel_length}" wheelRadius="${small_wheel_radius}" wheelMass="${small_wheel_weight}" meshFile="wheelchair_wheel_small"/>
-  <wheel_joint parent="front_right_leg_rev" child ="front_right_wheel" xyz="0.017 0 ${-0.07352}" rpy="0 0 0" axis="0 1 0"/>
+  <wheel_joint parent="front_right_leg_rev" child ="front_right_wheel" xyz="0.017 0 ${-2*small_wheel_radius + 0.0377}" rpy="0 0 0" axis="0 1 0"/>
 </robot>

File: src/wheelchair_description/urdf/wheelchair1.urdf (robot description, URDF)
Before this commit: robot wheelchair, 13 links, 12 joints
Links:
- removed link rear_left_leg
- removed link rear_right_leg
- added link base1, mass 0.1; collision box size=0.02 0.223568 0.15; visual box size=0.02 0.223568 0.15
- link base: geometry collision box size=0.250676 0.223568 0.01; visual box size=0.250676 0.223568 0.01
- link front_left_leg: geometry collision box size=0.01 0.01 0.0354; visual box size=0.01 0.01 0.0354
- link front_left_leg_rev: geometry collision cylinder length=0.01 radius=0.01; visual mesh filename=package://wheelchair_description/meshes/wheelchair_wheel_re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 scale=0.01 0.01 0.01
- link front_right_leg: geometry collision box size=0.01 0.01 0.0354; visual box size=0.01 0.01 0.0354
- link front_right_leg_rev: geometry collision cylinder length=0.01 radius=0.01; visual mesh filename=package://wheelchair_description/meshes/wheelchair_wheel_re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 scale=0.01 0.01 0.01
Joints:
- removed joint base_rear_left_leg_joint
- removed joint base_rear_right_leg_joint
- added joint axle_base1_joint: type fixed, parent axle, child base1, origin xyz=0 0 0 rpy=0 0 0
- joint axle_base_joint: origin xyz=0 0 0.1 rpy=0 0 0 -> xyz=0 0 0 rpy=0 0 0
- joint base_front_left_leg_joint: origin xyz=0.250676 0.161784 0 rpy=0 0 0 -> xyz=0.250676 0.111784 0 rpy=0 0 0
- joint base_front_right_leg_joint: origin xyz=0.250676 -0.161784 0 rpy=0 0 0 -> xyz=0.250676 -0.111784 0 rpy=0 0 0
- joint front_left_leg_front_left_leg_rev_joint: origin xyz=0 0 -0.16 rpy=0 0 0 -> xyz=0 0 -0.0354 rpy=0 0 0
- joint front_left_leg_rev_front_left_wheel_joint: origin xyz=0.017 0 -0.07352 rpy=0 0 0 -> xyz=0.04 0 -0.096 rpy=0 0 0
- joint front_right_leg_front_right_leg_rev_joint: origin xyz=0 0 -0.16 rpy=0 0 0 -> xyz=0 0 -0.0354 rpy=0 0 0
- joint front_right_leg_rev_front_right_wheel_joint: origin xyz=0.017 0 -0.07352 rpy=0 0 0 -> xyz=0.04 0 -0.096 rpy=0 0 0

File: src/wheelchair_description/urdf/wheelchair1.xacro (robot description, xacro)
@@ -3,5 +3,5 @@
   <xacro:property name="legs_width" value="0.01" />
   <xacro:property name="legs_length" value="0.01" />
-  <xacro:property name="legs_height" value="0.16" />
+  <xacro:property name="legs_height" value="0.0354" />
   <xacro:property name="legs_weight" value="0.25" />
   <xacro:property name="main_wheel_length" value="0.0356884" />
@@ -11,5 +11,5 @@
   <xacro:property name="small_wheel_length" value="0.032" />
   <xacro:property name="small_wheel_weight" value="1.5" />
-  <xacro:property name="chair_width" value="${2*main_wheel_radius - 0.08}" /> <!-- From front wheel right joint to front wheel left joint -->
+  <xacro:property name="chair_width" value="${2*main_wheel_radius - 0.18}" /> <!-- From front wheel right joint to front wheel left joint -->
   <xacro:property name="chair_length" value="${3/2*main_wheel_radius - 0.052}" /> 	 <!-- From front wheel joint to back wheel joint -->
   <xacro:property name="chair_height" value="0.01" /> 						 <!-- From front wheel joint to head rest -->
@@ -32,7 +32,7 @@
     <visual>
       <origin xyz="0 0 0" rpy="0 0 -3.14"/>
-      <geometry>
+      <!--geometry>
          <mesh filename="package://wheelchair_description/meshes/wheelchair_chasis.stl" scale="0.01 0.01 0.01"/>
-      </geometry>
+      </geometry-->
   </visual>
   </link>
@@ -58,16 +58,14 @@
   <link_joint parent="footprint" child ="axle" xyz="0 0 ${main_wheel_radius}" rpy="0 0 0" type="fixed"/>
   <chassis name="base" xyz="${chair_length/2} 0 0" rpy="0 0 0" m="${chair_weight}" chassisLength="${chair_length}" chassisWidth="${chair_width}" chassisHeight="${chair_height}"/>
-  <link_joint parent="axle" child ="base" xyz="0 0 0.1" rpy="0 0 0" type="fixed"/>
+  <link_joint parent="axle" child ="base" xyz="0 0 0" rpy="0 0 0" type="fixed"/>
+  <chassis name="base1" xyz="0 0 ${-0.15/2}" rpy="0 0 0" m="0.1" chassisLength="0.02" chassisWidth="${chair_width}" chassisHeight="0.15"/>
+  <link_joint parent="axle" child ="base1" xyz="0 0 0" rpy="0 0 0" type="fixed"/>
   <chassis name="front_left_leg" xyz="0 0 ${-legs_height/2}" rpy="0 0 0" m="${legs_weight}" chassisLength="${legs_length}" chassisWidth="${legs_width}" chassisHeight="${legs_height}"/>
   <link_joint parent="base" child ="front_left_leg" xyz="${chair_length} ${chair_width/2} 0" rpy="0 0 0" type="fixed"/>
-   <chassis name="rear_left_leg" xyz="0 0 ${-(legs_height + 0.1)/2}" rpy="0 0 0" m="${legs_weight}" chassisLength="${legs_length}" chassisWidth="${legs_width}" chassisHeight="${legs_height + 0.1}"/>
-  <link_joint parent="base" child ="rear_left_leg" xyz="0 ${chair_width/2} 0" rpy="0 0 0" type="fixed"/>
-<chassis name="rear_right_leg" xyz="0 0 ${-(legs_height + 0.1)/2}" rpy="0 0 0" m="${legs_weight}" chassisLength="${legs_length}" chassisWidth="${legs_width}" chassisHeight="${legs_height +0.1}"/>
-  <link_joint parent="base" child ="rear_right_leg" xyz="0 ${-chair_width/2} 0" rpy="0 0 0" type="fixed"/>
   <chassis name="front_right_leg" xyz="0 0 ${-legs_height/2}" rpy="0 0 0" m="${legs_weight}" chassisLength="${legs_length}" chassisWidth="${legs_width}" chassisHeight="${legs_height}"/>
   <link_joint parent="base" child ="front_right_leg" xyz="${chair_length} ${-chair_width/2} 0" rpy="0 0 0" type="fixed"/>
-  <wheel  lr="front_left_leg_rev" tY="0.02" xyz=" 0 0 0" rpy="0 0 0" wheelWidth="${0.1}" wheelRadius="${legs_width}" wheelMass="${legs_weight}" meshFile="wheelchair_wheel_rev"/>
+  <wheel  lr="front_left_leg_rev" tY="0.02" xyz=" 0 0 0" rpy="0 0 0" wheelWidth="${0.01}" wheelRadius="${legs_width}" wheelMass="${legs_weight}" meshFile="wheelchair_wheel_rev"/>
   <wheel_joint parent="front_left_leg" child ="front_left_leg_rev" xyz="0 0 ${-legs_height}" rpy="0 0 0" axis="0 0 1"/>
-  <wheel  lr="front_right_leg_rev" tY="0.02" xyz=" 0 0 0" rpy="0 0 0" wheelWidth="${0.1}" wheelRadius="${legs_width}" wheelMass="${legs_weight}" meshFile="wheelchair_wheel_rev"/>
+  <wheel  lr="front_right_leg_rev" tY="0.02" xyz=" 0 0 0" rpy="0 0 0" wheelWidth="${0.01}" wheelRadius="${legs_width}" wheelMass="${legs_weight}" meshFile="wheelchair_wheel_rev"/>
   <wheel_joint parent="front_right_leg" child ="front_right_leg_rev" xyz="0 0 ${-legs_height}" rpy="0 0 0" axis="0 0 1"/>
   <wheel  lr="rear_left_wheel" tY="0.02" xyz=" 0 0 0" rpy="${-pi/2} 0 0" wheelWidth="${main_wheel_length}" wheelRadius="${main_wheel_radius}" wheelMass="${main_wheel_weight}" meshFile="wheelchair_wheel"/>
@@ -76,6 +74,6 @@
   <wheel_joint parent="axle" child ="rear_right_wheel" xyz="0 ${-main_wheel_radius} 0" rpy="0 0 0" axis="0 1 0"/>
   <wheel  lr="front_left_wheel" tY="0.001" xyz=" 0 0 0" rpy="${pi/2} 0 0" wheelWidth="${small_wheel_length}" wheelRadius="${small_wheel_radius}" wheelMass="${small_wheel_weight}" meshFile="wheelchair_wheel_small"/>
-  <wheel_joint parent="front_left_leg_rev" child ="front_left_wheel" xyz="0.017 0 ${-0.07352}" rpy="0 0 0" axis="0 1 0"/>
+  <wheel_joint parent="front_left_leg_rev" child ="front_left_wheel" xyz="0.04 0 ${-2*small_wheel_radius+0.04}" rpy="0 0 0" axis="0 1 0"/>
   <wheel  lr="front_right_wheel" tY="0.001" xyz=" 0 0 0" rpy="${pi/2} 0 0" wheelWidth="${small_wheel_length}" wheelRadius="${small_wheel_radius}" wheelMass="${small_wheel_weight}" meshFile="wheelchair_wheel_small"/>
-  <wheel_joint parent="front_right_leg_rev" child ="front_right_wheel" xyz="0.017 0 ${-0.07352}" rpy="0 0 0" axis="0 1 0"/>
+  <wheel_joint parent="front_right_leg_rev" child ="front_right_wheel" xyz="0.04 0 ${-2*small_wheel_radius + 0.04}" rpy="0 0 0" axis="0 1 0"/>
 </robot>
