Commit message: video

File: src/mdu_description/urdf/mdu.xacro (robot description, xacro)
@@ -5,5 +5,5 @@
   <xacro:property name="main_wheel_weight" value="2.0" />
   <xacro:property name="axle_width" value="0.01" />
-  <xacro:property name="axle_length" value="${0.28}"/>
+  <xacro:property name="axle_length" value="${0.30}"/>
   <xacro:property name="axle_height" value="0.01" />
   <xacro:property name="axle_weight" value="2.0" />
@@ -59,6 +59,6 @@
   <link_joint parent='footprint' child='chassis' xyz="0 0 ${main_wheel_radius}" rpy="0 0 0" type="fixed"/>
   <wheel  lr="rear_left_wheel" tY="0.02" xyz=" 0 0 0" rpy="${-pi/2} 0 0" wheelWidth="${main_wheel_length}" wheelRadius="${main_wheel_radius}" wheelMass="${main_wheel_weight}" meshFile="wheelchair_wheel"/>
-  <wheel_joint parent="chassis" child ="rear_left_wheel" xyz="0.04 ${chassis_width/2 +0.02} 0" rpy="0 0 0" axis="0 1 0"/>
+  <wheel_joint parent="chassis" child ="rear_left_wheel" xyz="0.03 ${chassis_width/2 +0.02} 0" rpy="0 0 0" axis="0 1 0"/>
   <wheel  lr="rear_right_wheel" tY="0.02" xyz=" 0 0 0" rpy="${pi/2} 0 0" wheelWidth="${main_wheel_length}" wheelRadius="${main_wheel_radius}" wheelMass="${main_wheel_weight}" meshFile="wheelchair_wheel"/>
-  <wheel_joint parent="chassis" child ="rear_right_wheel" xyz="0.04 ${-chassis_width/2 - 0.02} 0" rpy="0 0 0" axis="0 1 0"/>
+  <wheel_joint parent="chassis" child ="rear_right_wheel" xyz="0.03 ${-chassis_width/2 - 0.02} 0" rpy="0 0 0" axis="0 1 0"/>
 </robot>
