Commit message: added person

File: src/mdu_description/urdf/mdu.urdf (robot description, URDF)
Before this commit: robot mdu, 4 links, 3 joints
Links:
- link chassis: mass 6.0 -> 20.0; geometry collision box size=0.3 0.2 0.2; collision sphere radius=0.0635
Joints:
- joint chassis_rear_left_wheel_joint: origin xyz=0.04 0.135 0 rpy=0 0 0 -> xyz=0.01 0.12 0 rpy=0 0 0
- joint chassis_rear_right_wheel_joint: origin xyz=0.04 -0.135 0 rpy=0 0 0 -> xyz=0.01 -0.12 0 rpy=0 0 0

File: src/mdu_description/urdf/mdu.xacro (robot description, xacro)
@@ -8,8 +8,8 @@
   <xacro:property name="axle_height" value="0.01" />
   <xacro:property name="axle_weight" value="2.0" />
-  <xacro:property name="chassis_width" value="${axle_length  - 0.05}" /> <!-- From front wheel right joint to front wheel left joint -->
+  <xacro:property name="chassis_width" value="${axle_length  - 0.1}" /> <!-- From front wheel right joint to front wheel left joint -->
   <xacro:property name="chassis_length" value="${chassis_width + 0.1}" /> 	 <!-- From front wheel joint to back wheel joint -->
-  <xacro:property name="chassis_height" value="0.1" /> 				 <!-- From front wheel joint to head rest -->
-  <xacro:property name="chassis_weight" value="${6.0}" />
+  <xacro:property name="chassis_height" value="0.2" /> 				 <!-- From front wheel joint to head rest -->
+  <xacro:property name="chassis_weight" value="${20.0}" />
   <xacro:include filename="$(find mdu_description)/urdf/mdu.gazebo" />
   <xacro:include filename="$(find mdu_description)/urdf/materials.xacro" />
@@ -59,6 +59,6 @@
   <link_joint parent='footprint' child='chassis' xyz="0 0 ${main_wheel_radius}" rpy="0 0 0" type="fixed"/>
   <wheel  lr="rear_left_wheel" tY="0.02" xyz=" 0 0 0" rpy="${-pi/2} 0 0" wheelWidth="${main_wheel_length}" wheelRadius="${main_wheel_radius}" wheelMass="${main_wheel_weight}" meshFile="wheelchair_wheel"/>
-  <wheel_joint parent="chassis" child ="rear_left_wheel" xyz="0.03 ${chassis_width/2 +0.02} 0" rpy="0 0 0" axis="0 1 0"/>
+  <wheel_joint parent="chassis" child ="rear_left_wheel" xyz="0.01 ${chassis_width/2 +0.02} 0" rpy="0 0 0" axis="0 1 0"/>
   <wheel  lr="rear_right_wheel" tY="0.02" xyz=" 0 0 0" rpy="${pi/2} 0 0" wheelWidth="${main_wheel_length}" wheelRadius="${main_wheel_radius}" wheelMass="${main_wheel_weight}" meshFile="wheelchair_wheel"/>
-  <wheel_joint parent="chassis" child ="rear_right_wheel" xyz="0.03 ${-chassis_width/2 - 0.02} 0" rpy="0 0 0" axis="0 1 0"/>
+  <wheel_joint parent="chassis" child ="rear_right_wheel" xyz="0.01 ${-chassis_width/2 - 0.02} 0" rpy="0 0 0" axis="0 1 0"/>
 </robot>

File: src/wheelchair_description/urdf/macros.xacro (robot description, xacro)
@@ -88,4 +88,34 @@
     </transmission>
   -->
+<xacro:macro name="sphere_" params="name xyz rpy m r">
+    <link name="${name}">
+      <collision name='${name}_collision'>
+        <geometry>
+        <sphere radius="${r}"/>
+	 </geometry>
+	<surface>
+	<friction>
+	  <ode>
+	    <mu>0</mu>
+	    <mu2>0</mu2>
+	    <slip1>0.0</slip1>
+	    <slip2>0.0</slip2>
+	  </ode>
+	</friction>
+	</surface>
+      </collision>
+      <visual name='${name}_visual'>
+        <origin xyz="${xyz}" rpy="${rpy}" />
+         <geometry>
+            <sphere radius="${r}"/>
+        </geometry>
+      </visual>
+      <inertial name="${name}_intertial">
+        <origin xyz="${xyz}" rpy="${rpy}" />
+        <mass value="${m}"/>
+        <sphere_inertia m="${m}" r ="${r}" />
+      </inertial>
+    </link>
+  </xacro:macro>
 <xacro:macro name="chassis" params="name xyz rpy m chassisLength chassisWidth chassisHeight">
     <link name="${name}">

File: src/wheelchair_description/urdf/wheelchair.urdf (robot description, URDF)
Before this commit: robot wheelchair, 13 links, 12 joints
Links:
- added link person_body, mass 60; collision sphere radius=0.161784; visual sphere radius=0.161784
- added link person_head, mass 5; collision sphere radius=0.080892; visual sphere radius=0.080892
Joints:
- added joint base_person_body_joint: type fixed, parent base, child person_body, origin xyz=0.161784 0 0.161784 rpy=0 0 0
- added joint person_body_person_head_joint: type fixed, parent person_body, child person_head, origin xyz=0 0 0.161784 rpy=0 0 0

File: src/wheelchair_description/urdf/wheelchair.xacro (robot description, xacro)
@@ -14,5 +14,5 @@
   <xacro:property name="chair_length" value="${3/2*main_wheel_radius - 0.052}" /> 	 <!-- From front wheel joint to back wheel joint -->
   <xacro:property name="chair_height" value="0.01" /> 						 <!-- From front wheel joint to head rest -->
-  <xacro:property name="chair_weight" value="${3.0+70.0}" />
+  <xacro:property name="chair_weight" value="${3.0}" />
   <xacro:property name="axle_width" value="0.01" />
   <xacro:property name="axle_length" value="${2*main_wheel_radius}"/>
@@ -79,3 +79,7 @@
   <wheel  lr="front_right_wheel" tY="0.001" xyz=" 0 0 0" rpy="${pi/2} 0 0" wheelWidth="${small_wheel_length}" wheelRadius="${small_wheel_radius}" wheelMass="${small_wheel_weight}" meshFile="wheelchair_wheel_small"/>
   <wheel_joint parent="front_right_leg_rev" child ="front_right_wheel" xyz="0.017 0 ${-0.07352}" rpy="0 0 0" axis="0 1 0"/>
+   <sphere_ name="person_body" xyz="0 0 0" rpy="0 0 0" m="60" r="${chair_width/2}"/>
+   <link_joint parent="base" child ="person_body" xyz="${chair_width/2} 0 ${chair_width/2}" rpy="0 0 0" type="fixed"/>
+   <sphere_ name="person_head" xyz="0 0 0" rpy="0 0 0" m="5" r="${chair_width/4}"/>
+   <link_joint parent="person_body" child ="person_head" xyz="0 0 ${chair_width/2}" rpy="0 0 0" type="fixed"/>
 </robot>
