Commit message: added transmission

File: src/mdu_description/urdf/macros.xacro (robot description, xacro)
@@ -56,34 +56,17 @@
         <cylinder_inertia m="${wheelMass}" r="${wheelRadius}" h="${wheelWidth}"/>
       </inertial>
+	    <!-- This block connects the wheel joint to an actuator (motor), which informs both
+		simulation and visualization of the robot -->
+		<transmission name="${lr}_wheel_trans">
+		  <type>transmission_interface/SimpleTransmission</type>
+		  <actuator name="${prefix}_${suffix}_wheel_motor">
+			<mechanicalReduction>1</mechanicalReduction>
+		  </actuator>
+		  <joint name="${prefix}_${suffix}_wheel_joint">
+			<hardwareInterface>VelocityJointInterface</hardwareInterface>
+		  </joint>
+		</transmission>
     </link>
   </xacro:macro>
-   <!--
-    <gazebo reference="${lr}_wheel">
-      <mu1 value="1.0"/>
-      <mu2 value="1.0"/>
-      <kp  value="10000000.0" />
-      <kd  value="1.0" />
-      <fdir1 value="1 0 0"/>
-      <material>Gazebo/Black</material>
-    </gazebo>
-    <joint name="${lr}_wheel_hinge" type="continuous">
-      <parent link="chassis"/>
-      <child link="${lr}_wheel"/>
-    <origin xyz="${-wheelPos+chassisLength/2} ${tY*wheelWidth/2+tY*chassisWidth/2} ${wheelRadius}" rpy="0 0 0" />
-      <axis xyz="0 1 0" rpy="0 0 0" />
-      <limit effort="10000" velocity="10000"/>
-      <joint_properties damping="0.0" friction="0.0"/>
-    </joint>
-    <transmission name="${lr}_trans">
-      <type>transmission_interface/SimpleTransmission</type>
-      <joint name="${lr}_wheel_hinge">
-        <hardwareInterface>EffortJointInterface</hardwareInterface>
-      </joint>
-      <actuator name="${lr}Motor">
-        <hardwareInterface>EffortJointInterface</hardwareInterface>
-        <mechanicalReduction>10</mechanicalReduction>
-      </actuator>
-    </transmission>
-  -->
 <xacro:macro name="chassis" params="name xyz rpy m chassisLength chassisWidth chassisHeight">
     <link name="${name}">

Commit message: merged

File: src/mdu_description/urdf/macros.xacro (robot description, xacro)
@@ -58,13 +58,13 @@
 	    <!-- This block connects the wheel joint to an actuator (motor), which informs both
 		simulation and visualization of the robot -->
-		<transmission name="${lr}_wheel_trans">
+		<!--transmission name="${lr}_wheel_trans">
 		  <type>transmission_interface/SimpleTransmission</type>
-		  <actuator name="${prefix}_${suffix}_wheel_motor">
+		  <actuator name="${lr}_wheel_motor">
 			<mechanicalReduction>1</mechanicalReduction>
 		  </actuator>
-		  <joint name="${prefix}_${suffix}_wheel_joint">
+		  <joint name="${lr}_motor_wheel_joint">
 			<hardwareInterface>VelocityJointInterface</hardwareInterface>
 		  </joint>
-		</transmission>
+		</transmission-->
     </link>
   </xacro:macro>

File: src/mdu_description/urdf/mdu.xacro (robot description, xacro)
@@ -1,25 +1,22 @@
 <?xml version='1.0'?>
 <robot name="mdu" xmlns:xacro="http://www.ros.org/wiki/xacro" >
-  <xacro:property name="main_wheel_length" value="0.0356884" />
+  <xacro:property name="main_wheel_length" value="0.05" />
   <xacro:property name="main_wheel_radius" value="0.127" />
   <xacro:property name="main_wheel_weight" value="3.0" />
   <xacro:property name="axle_width" value="0.01" />
-  <xacro:property name="axle_length" value="${2*main_wheel_radius}"/>
+  <xacro:property name="axle_length" value="${0.28}"/>
   <xacro:property name="axle_height" value="0.01" />
   <xacro:property name="axle_weight" value="2.0" />
-  <xacro:property name="chair_width" value="${axle_length  - 0.5}" /> <!-- From front wheel right joint to front wheel left joint -->
-  <xacro:property name="chair_length" value="${chair_width}" /> 	 <!-- From front wheel joint to back wheel joint -->
-  <xacro:property name="chair_height" value="0.05" /> 				 <!-- From front wheel joint to head rest -->
+  <xacro:property name="chair_width" value="${axle_length  - 0.05}" /> <!-- From front wheel right joint to front wheel left joint -->
+  <xacro:property name="chair_length" value="${chair_width - 0.1}" /> 	 <!-- From front wheel joint to back wheel joint -->
+  <xacro:property name="chair_height" value="0.15" /> 				 <!-- From front wheel joint to head rest -->
   <xacro:property name="chair_weight" value="${10.0}" />
-  <xacro:include filename="$(find wheelchair_description)/urdf/mdu.gazebo" />
-  <xacro:include filename="$(find wheelchair_description)/urdf/materials.xacro" />
-  <xacro:include filename="$(find wheelchair_description)/urdf/macros.xacro" />
+  <xacro:include filename="$(find mdu_description)/urdf/mdu.gazebo" />
+  <xacro:include filename="$(find mdu_description)/urdf/materials.xacro" />
+  <xacro:include filename="$(find mdu_description)/urdf/macros.xacro" />
   <link name='footprint'>
-	<pose xyz="-10 0 0" rpy=" 0 0 0"/>
+    <pose xyz="0 0 0" rpy=" 0 0 0"/>
     <visual>
       <origin xyz="0 0 0" rpy=" 0 0 0"/>
-    <geometry>
-      <box size="0.001 0.001 0.001"/>
-    </geometry>
     </visual>
     <!--visual>
@@ -49,10 +46,35 @@
     </visual>
   </link>
+  <link name='caster'>
+      <collision name='caster_collision'>
+	      <origin xyz="0 0 0" rpy=" 0 0 0"/>
+	      <geometry>
+		<sphere radius="${main_wheel_radius/2}"/>
+	      </geometry>
+	      <surface>
+		<friction>
+		  <ode>
+		    <mu>0</mu>
+		    <mu2>0</mu2>
+		    <slip1>1.0</slip1>
+		    <slip2>1.0</slip2>
+		  </ode>
+		</friction>
+	      </surface>
+    </collision>
+    <visual name='caster_visual'>
+      <origin xyz="0 0 0" rpy=" 0 0 0"/>
+      <geometry>
+        <sphere radius="${main_wheel_radius/2}"/>
+      </geometry>
+   </visual>
+ </link>
   <link_joint parent="footprint" child ="axle" xyz="0 0 ${main_wheel_radius}" rpy="0 0 0" type="fixed"/>
   <chassis name="base" xyz="${chair_length/2} 0 0" rpy="0 0 0" m="${chair_weight}" chassisLength="${chair_length}" chassisWidth="${chair_width}" chassisHeight="${chair_height}"/>
   <link_joint parent="axle" child ="base" xyz="0 0 0" rpy="0 0 0" type="fixed"/>
+  <link_joint parent="base" child ="caster" xyz="${chair_length -main_wheel_radius/2} 0 ${-main_wheel_radius/2}" rpy="0 0 0" type="fixed"/>
   <wheel  lr="rear_left_wheel" tY="0.02" xyz=" 0 0 0" rpy="${-pi/2} 0 0" wheelWidth="${main_wheel_length}" wheelRadius="${main_wheel_radius}" wheelMass="${main_wheel_weight}" meshFile="wheelchair_wheel"/>
-  <wheel_joint parent="axle" child ="rear_left_wheel" xyz="0 ${main_wheel_radius} 0" rpy="0 0 0" axis="0 1 0"/>
+  <wheel_joint parent="axle" child ="rear_left_wheel" xyz="0 ${axle_length/2} 0" rpy="0 0 0" axis="0 1 0"/>
   <wheel  lr="rear_right_wheel" tY="0.02" xyz=" 0 0 0" rpy="${pi/2} 0 0" wheelWidth="${main_wheel_length}" wheelRadius="${main_wheel_radius}" wheelMass="${main_wheel_weight}" meshFile="wheelchair_wheel"/>
-  <wheel_joint parent="axle" child ="rear_right_wheel" xyz="0 ${-main_wheel_radius} 0" rpy="0 0 0" axis="0 1 0"/>
+  <wheel_joint parent="axle" child ="rear_right_wheel" xyz="0 ${-axle_length/2} 0" rpy="0 0 0" axis="0 1 0"/>
 </robot>

File: src/wheelchair_description/urdf/wheelchair.urdf (robot description, URDF)
Before this commit: robot wheelchair, 11 links, 10 joints
Links:
- removed link rl_wheel
- removed link rr_wheel
- added link base1, mass 5; collision box size=0.02 0.223568 0.15; visual box size=0.02 0.223568 0.15
- added link rear_left_wheel, mass 3.0; collision cylinder length=0.0356884 radius=0.201784; visual mesh filename=package://wheelchair_description/meshes/wheelchair_wheel.stl scale=0.01 0.01 0.01
- added link rear_right_wheel, mass 3.0; collision cylinder length=0.0356884 radius=0.201784; visual mesh filename=package://wheelchair_description/meshes/wheelchair_wheel.stl scale=0.01 0.01 0.01
- link base: mass 3.0 -> 73.0
Joints:
- removed joint axle_rl_wheel_joint
- removed joint axle_rr_wheel_joint
- added joint axle_base1_joint: type fixed, parent axle, child base1, origin xyz=0 0 0 rpy=0 0 0
- added joint axle_rear_left_wheel_joint: type continuous, parent axle, child rear_left_wheel, origin xyz=0 0.201784 0 rpy=0 0 0, axis 0 1 0, limit effort=100 velocity=100
- added joint axle_rear_right_wheel_joint: type continuous, parent axle, child rear_right_wheel, origin xyz=0 -0.201784 0 rpy=0 0 0, axis 0 1 0, limit effort=100 velocity=100

File: src/wheelchair_description/urdf/wheelchair.xacro (robot description, xacro)
@@ -23,4 +23,5 @@
   <xacro:include filename="$(find wheelchair_description)/urdf/macros.xacro" />
   <link name='footprint'>
+    <pose xyz="10 0 0" rpy=" 0 0 0"/>
     <visual>
       <origin xyz="0 0 0" rpy=" 0 0 0"/>
@@ -58,4 +59,6 @@
   <chassis name="base" xyz="${chair_length/2} 0 0" rpy="0 0 0" m="${chair_weight}" chassisLength="${chair_length}" chassisWidth="${chair_width}" chassisHeight="${chair_height}"/>
   <link_joint parent="axle" child ="base" xyz="0 0 0" rpy="0 0 0" type="fixed"/>
+  <chassis name="base1" xyz="0 0 ${-0.15/2}" rpy="0 0 0" m="0.1" chassisLength="0.02" chassisWidth="${chair_width}" chassisHeight="0.15"/>
+  <link_joint parent="axle" child ="base1" xyz="0 0 0" rpy="0 0 0" type="fixed"/>
   <chassis name="front_left_leg" xyz="0 0 ${-legs_height/2}" rpy="0 0 0" m="${legs_weight}" chassisLength="${legs_length}" chassisWidth="${legs_width}" chassisHeight="${legs_height}"/>
   <link_joint parent="base" child ="front_left_leg" xyz="${chair_length} ${chair_width/2} 0" rpy="0 0 0" type="fixed"/>
