Commit message: added pictures

File: src/mdu_description/urdf/macros.xacro (robot description, xacro)
@@ -29,5 +29,5 @@
     </joint>
   </xacro:macro>
-  <xacro:macro name="wheel" params="lr tY xyz rpy wheelWidth wheelRadius wheelMass meshFile">
+  <xacro:macro name="wheel_mdu" params="lr tY xyz rpy wheelWidth wheelRadius wheelMass meshFile">
     <link name="${lr}">
       <collision name="${lr}_collision">
@@ -69,4 +69,21 @@
     </link>
   </xacro:macro>
+ <xacro:macro name="wheel__mdu" params="lr tY xyz rpy wheelWidth wheelRadius wheelMass meshFile">
+    <link name="${lr}">
+      <visual name="${lr}_visual">
+        <transparency>0.1</transparency>
+        <origin xyz="${xyz}" rpy="${rpy}" />
+        <geometry>
+          <cylinder length="${wheelWidth - tY}" radius="${wheelRadius}"/>
+        </geometry>
+        <material name="green"/>
+      </visual>
+      <inertial name="${lr}_visual_intertial">
+        <origin xyz="0 0 0" rpy="0 ${pi/2} ${pi/2}" />
+        <mass value="${wheelMass}"/>
+        <cylinder_inertia m="${wheelMass}" r="${wheelRadius}" h="${wheelWidth}"/>
+      </inertial>
+    </link>
+  </xacro:macro>
 <xacro:macro name="chassis" params="name xyz rpy m chassisLength chassisWidth chassisHeight">
     <link name="${name}">

File: src/mdu_description/urdf/mdu.urdf (robot description, URDF)
Before this commit: robot mdu, 4 links, 3 joints
Links:
- removed link footprint
- removed link rear_left_wheel
- removed link rear_right_wheel
- added link front_left_pipe, mass 0.5; collision cylinder length=0.01 radius=0.015; visual cylinder length=0.009 radius=0.015
- added link front_right_pipe, mass 0.5; collision cylinder length=0.01 radius=0.015; visual cylinder length=0.009 radius=0.015
- added link rear_left_wheel_mdu, mass 2.0; collision cylinder length=0.05 radius=0.127; visual cylinder length=0.03 radius=0.127
- added link rear_right_wheel_mdu, mass 2.0; collision cylinder length=0.05 radius=0.127; visual cylinder length=0.03 radius=0.127
- link chassis: mass 20.0 -> 15.0; geometry collision box size=0.43 0.25 0.2; collision sphere radius=0.0635
Joints:
- removed joint chassis_rear_left_wheel_joint
- removed joint chassis_rear_right_wheel_joint
- removed joint footprint_chassis_joint
- added joint chassis_rear_left_wheel_mdu_joint: type continuous, parent chassis, child rear_left_wheel_mdu, origin xyz=0.05 0.145 0 rpy=0 0 0, axis 0 1 0, limit effort=100 velocity=100
- added joint chassis_rear_right_wheel_mdu_joint: type continuous, parent chassis, child rear_right_wheel_mdu, origin xyz=0.05 -0.145 0 rpy=0 0 0, axis 0 1 0, limit effort=100 velocity=100
- added joint front_left_pipe_chassis_joint: type fixed, parent front_left_pipe, child chassis, origin xyz=-0.215 -0.065 0.0848 rpy=0 0 0

File: src/mdu_description/urdf/mdu.xacro (robot description, xacro)
@@ -1,27 +1,27 @@
 <?xml version='1.0'?>
 <robot name="mdu" xmlns:xacro="http://www.ros.org/wiki/xacro" >
-  <xacro:property name="main_wheel_length" value="0.05" />
-  <xacro:property name="main_wheel_radius" value="0.127" />
-  <xacro:property name="main_wheel_weight" value="2.0" />
-  <xacro:property name="axle_width" value="0.01" />
-  <xacro:property name="axle_length" value="${0.30}"/>
-  <xacro:property name="axle_height" value="0.01" />
-  <xacro:property name="axle_weight" value="2.0" />
-  <xacro:property name="chassis_width" value="${axle_length  - 0.1}" /> <!-- From front wheel right joint to front wheel left joint -->
-  <xacro:property name="chassis_length" value="${chassis_width + 0.1}" /> 	 <!-- From front wheel joint to back wheel joint -->
-  <xacro:property name="chassis_height" value="0.2" /> 				 <!-- From front wheel joint to head rest -->
-  <xacro:property name="chassis_weight" value="${20.0}" />
+  <xacro:property name="main_wheel_length_mdu" value="0.05" />
+  <xacro:property name="main_wheel_radius_mdu" value="0.127" />
+  <xacro:property name="main_wheel_weight_mdu" value="2.0" />
+  <xacro:property name="axle_width_mdu" value="0.01" />
+  <xacro:property name="axle_length_mdu" value="${0.30}"/>
+  <xacro:property name="axle_height_mdu" value="0.01" />
+  <xacro:property name="axle_weight_mdu" value="0.1" />
+  <xacro:property name="chassis_width_mdu" value="${axle_length_mdu  - 0.05}" /> <!-- From front wheel right joint to front wheel left joint -->
+ <xacro:property name="chassis_width__mdu" value="${0.33 }" /> <!-- From front wheel right joint to front wheel left joint -->
+  <xacro:property name="chassis_length_mdu" value="${chassis_width__mdu +0.1}" /> 	 <!-- From front wheel joint to back wheel joint -->
+  <xacro:property name="chassis_height_mdu" value="0.2" /> 				 <!-- From front wheel joint to head rest -->
+  <xacro:property name="chassis_weight_mdu" value="${15.0}" />
   <xacro:include filename="$(find mdu_description)/urdf/mdu.gazebo" />
-  <xacro:include filename="$(find mdu_description)/urdf/materials.xacro" />
   <xacro:include filename="$(find mdu_description)/urdf/macros.xacro" />
   <link name='chassis'>
     <inertial name="chassis_intertial">
         <origin xyz="0 0 0" rpy="0 0 0" />
-        <mass value="${chassis_weight}"/>
-        <box_inertia m="${chassis_weight}" x="${chassis_length}" y="${chassis_width}" z ="${chassis_height}" />
+        <mass value="${chassis_weight_mdu}"/>
+        <box_inertia m="${chassis_weight_mdu}" x="${chassis_length_mdu}" y="${chassis_width_mdu}" z ="${chassis_height_mdu}" />
       </inertial>
     <collision name='collision'>
       <geometry>
-        <box size="${chassis_length} ${chassis_width} ${chassis_height}"/>
+        <box size="${chassis_length_mdu} ${chassis_width_mdu} ${chassis_height_mdu}"/>
       </geometry>
     </collision>
@@ -29,17 +29,17 @@
       <origin xyz="0 0 0" rpy="0 0 0" />
       <geometry>
-        <box size="${chassis_length} ${chassis_width} ${chassis_height}"/>
+        <box size="${chassis_length_mdu} ${chassis_width_mdu} ${chassis_height_mdu}"/>
       </geometry>
     </visual>
     <collision name='caster_collision'>
-      <origin xyz="${-(chassis_length/2 - (main_wheel_radius/2))} 0 ${-main_wheel_radius/2}" rpy=" 0 0 0"/>
+      <origin xyz="${-(chassis_length_mdu/2 - main_wheel_radius_mdu/2)} 0 ${-main_wheel_radius_mdu/2}" rpy=" 0 0 0"/>
       <geometry>
-        <sphere radius="${(main_wheel_radius/2)}"/>
+        <sphere radius="${(main_wheel_radius_mdu/2)}"/>
       </geometry>
       <surface>
         <friction>
           <ode>
-            <mu>0</mu>
-            <mu2>0</mu2>
+            <mu>0.5</mu>
+            <mu2>0.5</mu2>
             <slip1>1.0</slip1>
             <slip2>1.0</slip2>
@@ -49,16 +49,20 @@
     </collision>
     <visual name='caster_visual'>
-      <origin xyz="${-(chassis_length/2 - (main_wheel_radius/2))} 0 ${-main_wheel_radius/2}" rpy=" 0 0 0"/>
+      <origin xyz="${-(chassis_length_mdu/2 - main_wheel_radius_mdu/2)} 0 ${-main_wheel_radius_mdu/2}" rpy=" 0 0 0"/>
       <geometry>
-        <sphere radius="${(main_wheel_radius/2)}"/>
+        <sphere radius="${(main_wheel_radius_mdu/2)}"/>
       </geometry>
     </visual>
   </link>
-  <link name='footprint'>
-  </link>
-  <link_joint parent='footprint' child='chassis' xyz="0 0 ${main_wheel_radius}" rpy="0 0 0" type="fixed"/>
-  <wheel  lr="rear_left_wheel" tY="0.02" xyz=" 0 0 0" rpy="${-pi/2} 0 0" wheelWidth="${main_wheel_length}" wheelRadius="${main_wheel_radius}" wheelMass="${main_wheel_weight}" meshFile="wheelchair_wheel"/>
-  <wheel_joint parent="chassis" child ="rear_left_wheel" xyz="0.01 ${chassis_width/2 +0.02} 0" rpy="0 0 0" axis="0 1 0"/>
-  <wheel  lr="rear_right_wheel" tY="0.02" xyz=" 0 0 0" rpy="${pi/2} 0 0" wheelWidth="${main_wheel_length}" wheelRadius="${main_wheel_radius}" wheelMass="${main_wheel_weight}" meshFile="wheelchair_wheel"/>
-  <wheel_joint parent="chassis" child ="rear_right_wheel" xyz="0.01 ${-chassis_width/2 - 0.02} 0" rpy="0 0 0" axis="0 1 0"/>
+  <!--link name='footprint_mdu'>
+  </link-->
+  <!--link_joint parent='footprint_mdu' child='chassis' xyz="0 0 ${main_wheel_radius_mdu}" rpy="0 0 0" type="fixed"/-->
+  <wheel_mdu  lr="rear_left_wheel_mdu" tY="0.02" xyz=" 0 0 0" rpy="${-pi/2} 0 0" wheelWidth="${main_wheel_length_mdu}" wheelRadius="${main_wheel_radius_mdu}" wheelMass="${main_wheel_weight_mdu}" meshFile="wheelchair_wheel"/>
+  <wheel_joint parent="chassis" child ="rear_left_wheel_mdu" xyz="0.05 ${chassis_width_mdu/2 +0.02} 0" rpy="0 0 0" axis="0 1 0"/>
+  <wheel_mdu  lr="rear_right_wheel_mdu" tY="0.02" xyz=" 0 0 0" rpy="${pi/2} 0 0" wheelWidth="${main_wheel_length_mdu}" wheelRadius="${main_wheel_radius_mdu}" wheelMass="${main_wheel_weight_mdu}" meshFile="wheelchair_wheel"/>
+  <wheel_joint parent="chassis" child ="rear_right_wheel_mdu" xyz="0.05 ${-chassis_width_mdu/2 - 0.02} 0" rpy="0 0 0" axis="0 1 0"/>
+  <wheel_mdu  lr="front_right_pipe" tY="0.001" xyz=" 0 0 0" rpy="0 ${pi/2} 0" wheelWidth="${0.01}" wheelRadius="${0.015}" wheelMass="${0.5}" meshFile="pipe"/>
+  <!--link_joint parent='front_right_pipe' child='chassis' xyz="${chassis_length_mdu/2 } ${chassis_width__mdu/2 - 0.10} ${(0.082 + 0.00280)}" rpy="0 0 0" type="fixed"/-->
+  <wheel_mdu  lr="front_left_pipe" tY="0.001" xyz=" 0 0 0" rpy="0 ${pi/2} 0" wheelWidth="${0.01}" wheelRadius="${0.015}" wheelMass="${0.5}" meshFile="pipe"/>
+  <link_joint parent='front_left_pipe' child='chassis' xyz="${-chassis_length_mdu/2 } ${-chassis_width__mdu/2 +0.10} ${0.082 + 0.00280}" rpy="0 0 0" type="fixed"/>
 </robot>

File: src/wheelchair_description/urdf/macros.xacro (robot description, xacro)
@@ -34,9 +34,8 @@
         <origin xyz="${xyz}" rpy="${rpy}" />
         <geometry>
-          <cylinder length="${wheelWidth}" radius="${wheelRadius}"/>
+          <mesh filename="package://wheelchair_description/meshes/${meshFile}.stl" scale="0.01 0.01 0.01"/>
         </geometry>
       </collision>
-      <!--
-      <visual name="${lr}_visual">
+      <!--visual name="${lr}_visual">
         <transparency>0.1</transparency>
         <origin xyz="${xyz}" rpy="${rpy}" />
@@ -45,6 +44,20 @@
         </geometry>
         <material name="green"/>
+      </visual-->
+      <visual name="${lr}_visual_mesh">
+        <origin xyz="${xyz}" rpy="${rpy}" />
+        <geometry>
+          <mesh filename="package://wheelchair_description/meshes/${meshFile}.stl" scale="0.01 0.01 0.01"/>
+        </geometry>
       </visual>
-    -->
+      <inertial name="${lr}_visual_intertial">
+        <origin xyz="0 0 0" rpy="0 ${pi/2} ${pi/2}" />
+        <mass value="${wheelMass}"/>
+        <cylinder_inertia m="${wheelMass}" r="${wheelRadius}" h="${wheelWidth}"/>
+      </inertial>
+    </link>
+  </xacro:macro>
+  <xacro:macro name="wheel_" params="lr tY xyz rpy wheelWidth wheelRadius wheelMass meshFile">
+    <link name="${lr}">
       <visual name="${lr}_visual_mesh">
         <origin xyz="${xyz}" rpy="${rpy}" />
@@ -97,6 +110,6 @@
 	<friction>
 	  <ode>
-	    <mu>0</mu>
-	    <mu2>0</mu2>
+	    <mu>0.5</mu>
+	    <mu2>0.5</mu2>
 	    <slip1>0.0</slip1>
 	    <slip2>0.0</slip2>

File: src/wheelchair_description/urdf/wheelchair.urdf (robot description, URDF)
Before this commit: robot wheelchair, 15 links, 14 joints
Links:
- added link chassis, mass 15.0; collision box size=0.43 0.25 0.2; collision sphere radius=0.0635
- added link front_left_pipe, mass 0.5; collision cylinder length=0.01 radius=0.015; visual cylinder length=0.009 radius=0.015
- added link front_right_pipe, mass 0.5; collision cylinder length=0.01 radius=0.015; visual cylinder length=0.009 radius=0.015
- added link rear_left_pipe, mass 0.5; collision mesh filename=package://wheelchair_description/meshes/pipe.stl scale=0.01 0.01 0.01; visual mesh filename=package://wheelchair_description/meshes/pipe.stl scale=0.01 0.01 0.01
- added link rear_left_wheel_mdu, mass 2.0; collision cylinder length=0.05 radius=0.127; visual cylinder length=0.03 radius=0.127
- added link rear_right_pipe, mass 0.5; collision mesh filename=package://wheelchair_description/meshes/pipe.stl scale=0.01 0.01 0.01; visual mesh filename=package://wheelchair_description/meshes/pipe.stl scale=0.01 0.01 0.01
- added link rear_right_wheel_mdu, mass 2.0; collision cylinder length=0.05 radius=0.127; visual cylinder length=0.03 radius=0.127
- link base: mass 73.0 -> 3.0
- link front_left_leg_rev: geometry collision mesh filename=package://wheelchair_description/meshes/wheelchair_wheel_re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 scale=0.01 0.01 0.01; visual mesh filename=package://wheelchair_description/meshes/wheelchair_wheel_re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 scale=0.01 0.01 0.01
- link front_left_wheel: geometry collision mesh filename=package://wheelchair_description/meshes/wheelchair_wheel_sm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 scale=0.01 0.01 0.01; visual mesh filename=package://wheelchair_description/meshes/wheelchair_wheel_sm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 scale=0.01 0.01 0.01
- link front_right_leg_rev: geometry collision mesh filename=package://wheelchair_description/meshes/wheelchair_wheel_re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 scale=0.01 0.01 0.01; visual mesh filename=package://wheelchair_description/meshes/wheelchair_wheel_re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 scale=0.01 0.01 0.01
- link front_right_wheel: geometry collision mesh filename=package://wheelchair_description/meshes/wheelchair_wheel_sm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 scale=0.01 0.01 0.01; visual mesh filename=package://wheelchair_description/meshes/wheelchair_wheel_sm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 scale=0.01 0.01 0.01
- link person_body: mass 60 -> 65; geometry collision sphere radius=0.141784; visual sphere radius=0.141784
- link rear_left_wheel: geometry collision mesh filename=package://wheelchair_description/meshes/wheelchair_wheel.stl scale=0.01 0.01 0.01; visual mesh filename=package://wheelchair_description/meshes/wheelchair_wheel.stl scale=0.01 0.01 0.01
- link rear_right_wheel: geometry collision mesh filename=package://wheelchair_description/meshes/wheelchair_wheel.stl scale=0.01 0.01 0.01; visual mesh filename=package://wheelchair_description/meshes/wheelchair_wheel.stl scale=0.01 0.01 0.01
Joints:
- added joint chassis_rear_left_wheel_mdu_joint: type continuous, parent chassis, child rear_left_wheel_mdu, origin xyz=0.05 0.145 0 rpy=0 0 0, axis 0 1 0, limit effort=100 velocity=100
- added joint chassis_rear_right_wheel_mdu_joint: type continuous, parent chassis, child rear_right_wheel_mdu, origin xyz=0.05 -0.145 0 rpy=0 0 0, axis 0 1 0, limit effort=100 velocity=100
- added joint front_left_pipe_chassis_joint: type fixed, parent front_left_pipe, child chassis, origin xyz=-0.215 -0.065 0.0848 rpy=0 0 0
- added joint rear_left_leg_rear_left_pipe_joint: type fixed, parent rear_left_leg, child rear_left_pipe, origin xyz=0 0 -0.26 rpy=0 0 0
- added joint rear_left_pipe_front_left_pipe_joint: type fixed, parent rear_left_pipe, child front_left_pipe, origin xyz=0 0 0 rpy=0 0 0
- added joint rear_right_leg_rear_right_pipe_joint: type fixed, parent rear_right_leg, child rear_right_pipe, origin xyz=0 0 -0.26 rpy=0 0 0
- added joint rear_right_pipe_front_right_pipe_joint: type fixed, parent rear_right_pipe, child front_right_pipe, origin xyz=0 0 0 rpy=0 0 0
- joint base_person_body_joint: origin xyz=0.161784 0 0.161784 rpy=0 0 0 -> xyz=0.141784 0 0.141784 rpy=0 0 0
- joint base_rear_left_leg_joint: origin xyz=0 0.161784 0 rpy=0 0 0 -> xyz=0 0.061784 0 rpy=0 0 0
- joint base_rear_right_leg_joint: origin xyz=0 -0.161784 0 rpy=0 0 0 -> xyz=0 -0.061784 0 rpy=0 0 0

File: src/wheelchair_description/urdf/wheelchair.xacro (robot description, xacro)
@@ -22,4 +22,5 @@
   <xacro:include filename="$(find wheelchair_description)/urdf/materials.xacro" />
   <xacro:include filename="$(find wheelchair_description)/urdf/macros.xacro" />
+  <xacro:include filename="$(find mdu_description)/urdf/mdu.xacro" />
   <link name='footprint'>
     <pose xyz="1 0 0" rpy=" 0 0 0"/>
@@ -62,7 +63,7 @@
   <link_joint parent="base" child ="front_left_leg" xyz="${chair_length} ${chair_width/2} 0" rpy="0 0 0" type="fixed"/>
    <chassis name="rear_left_leg" xyz="0 0 ${-(legs_height + 0.1)/2}" rpy="0 0 0" m="${legs_weight}" chassisLength="${legs_length}" chassisWidth="${legs_width}" chassisHeight="${legs_height + 0.1}"/>
-  <link_joint parent="base" child ="rear_left_leg" xyz="0 ${chair_width/2} 0" rpy="0 0 0" type="fixed"/>
+  <link_joint parent="base" child ="rear_left_leg" xyz="0 ${chair_width/2 - 0.1} 0" rpy="0 0 0" type="fixed"/>
 <chassis name="rear_right_leg" xyz="0 0 ${-(legs_height + 0.1)/2}" rpy="0 0 0" m="${legs_weight}" chassisLength="${legs_length}" chassisWidth="${legs_width}" chassisHeight="${legs_height +0.1}"/>
-  <link_joint parent="base" child ="rear_right_leg" xyz="0 ${-chair_width/2} 0" rpy="0 0 0" type="fixed"/>
+  <link_joint parent="base" child ="rear_right_leg" xyz="0 ${-chair_width/2 + 0.1} 0" rpy="0 0 0" type="fixed"/>
   <chassis name="front_right_leg" xyz="0 0 ${-legs_height/2}" rpy="0 0 0" m="${legs_weight}" chassisLength="${legs_length}" chassisWidth="${legs_width}" chassisHeight="${legs_height}"/>
   <link_joint parent="base" child ="front_right_leg" xyz="${chair_length} ${-chair_width/2} 0" rpy="0 0 0" type="fixed"/>
@@ -79,7 +80,13 @@
   <wheel  lr="front_right_wheel" tY="0.001" xyz=" 0 0 0" rpy="${pi/2} 0 0" wheelWidth="${small_wheel_length}" wheelRadius="${small_wheel_radius}" wheelMass="${small_wheel_weight}" meshFile="wheelchair_wheel_small"/>
   <wheel_joint parent="front_right_leg_rev" child ="front_right_wheel" xyz="0.017 0 ${-0.07352}" rpy="0 0 0" axis="0 1 0"/>
-   <sphere_ name="person_body" xyz="0 0 0" rpy="0 0 0" m="60" r="${chair_width/2}"/>
-   <link_joint parent="base" child ="person_body" xyz="${chair_width/2} 0 ${chair_width/2}" rpy="0 0 0" type="fixed"/>
+   <sphere_ name="person_body" xyz="0 0 0" rpy="0 0 0" m="65" r="${chair_width/2 -0.02}"/>
+   <link_joint parent="base" child ="person_body" xyz="${chair_width/2 -0.02} 0 ${chair_width/2 -0.02}" rpy="0 0 0" type="fixed"/>
    <sphere_ name="person_head" xyz="0 0 0" rpy="0 0 0" m="5" r="${chair_width/4}"/>
    <link_joint parent="person_body" child ="person_head" xyz="0 0 ${chair_width/2}" rpy="0 0 0" type="fixed"/>
+   <wheel  lr="rear_right_pipe" tY="0.001" xyz=" ${-0.025} 0 -0.01" rpy="0 ${pi/2} 0" wheelWidth="${0.05}" wheelRadius="${0.04}" wheelMass="${0.5}" meshFile="pipe"/>
+   <link_joint parent="rear_right_leg" child ="rear_right_pipe" xyz="0 0 ${-legs_height-0.1}" rpy="0 0 0" type="fixed"/>
+   <wheel  lr="rear_left_pipe" tY="0.001" xyz=" ${-0.025} 0 -0.01" rpy="0 ${pi/2} 0" wheelWidth="${0.05}" wheelRadius="${0.04}" wheelMass="${0.5}" meshFile="pipe"/>
+   <link_joint parent="rear_left_leg" child ="rear_left_pipe" xyz="0 0 ${-legs_height-0.1}" rpy="0 0 0" type="fixed"/>
+    <link_joint parent="rear_left_pipe" child ="front_left_pipe" xyz="0 0 0" rpy="0 0 0" type="fixed"/>
+    <link_joint parent="rear_right_pipe" child ="front_right_pipe" xyz="0 0 0" rpy="0 0 0" type="fixed"/>
 </robot>
