Commit message: updated mdu design

File: src/mdu_description/urdf/macros.xacro (robot description, xacro)
@@ -113,3 +113,30 @@
     </joint>
   </xacro:macro>
+  <xacro:macro name="link_" params="name xyz rpy m length width height">
+      <link name="${name}">
+        <collision name='${name}_link_collision'>
+          <geometry>
+            <box size="${length} ${width} ${height}"/>
+          </geometry>
+        </collision>
+        <visual name='${name}_visual'>
+          <origin xyz="${xyz}" rpy="${rpy}" />
+            <geometry>
+              <box size="${length} ${width} ${height}"/>
+          </geometry>
+        </visual>
+        <inertial name="${name}_intertial">
+          <origin xyz="${xyz}" rpy="${rpy}" />
+          <mass value="${m}"/>
+          <box_inertia m="${m}" x="${length}" y="${width}" z ="${height}" />
+        </inertial>
+      </link>
+    </xacro:macro>
+    <xacro:macro name="link_joint" params="parent child xyz rpy type">
+      <joint type="${type}" name="${parent}_${child}_joint">
+        <origin xyz="${xyz}" rpy="${rpy}"/>
+        <parent link="${parent}"/>
+        <child link="${child}"/>
+      </joint>
+    </xacro:macro>
 </robot>

File: src/mdu_description/urdf/mdu.xacro (robot description, xacro)
@@ -2,14 +2,14 @@
 <robot name="mdu" xmlns:xacro="http://www.ros.org/wiki/xacro" >
   <xacro:property name="main_wheel_length_mdu" value="0.05" />
-  <xacro:property name="main_wheel_radius_mdu" value="0.127" />
+  <xacro:property name="main_wheel_radius_mdu" value="0.08255" /> <!--0.127-->
   <xacro:property name="main_wheel_weight_mdu" value="2.0" />
   <xacro:property name="axle_width_mdu" value="0.01" />
-  <xacro:property name="axle_length_mdu" value="${0.30}"/>
+  <xacro:property name="axle_length_mdu" value="${0.2}"/> <!-- 0.03-->
   <xacro:property name="axle_height_mdu" value="0.01" />
   <xacro:property name="axle_weight_mdu" value="0.1" />
   <xacro:property name="chassis_width_mdu" value="${axle_length_mdu  - 0.05}" /> <!-- From front wheel right joint to front wheel left joint -->
- <xacro:property name="chassis_width__mdu" value="${0.33 }" /> <!-- From front wheel right joint to front wheel left joint -->
-  <xacro:property name="chassis_length_mdu" value="${chassis_width__mdu +0.1}" /> 	 <!-- From front wheel joint to back wheel joint -->
-  <xacro:property name="chassis_height_mdu" value="0.2" /> 				 <!-- From front wheel joint to head rest -->
+ <xacro:property name="chassis_width__mdu" value="${chassis_width_mdu}" /> <!-- From front wheel right joint to front wheel left joint -->
+  <xacro:property name="chassis_length_mdu" value="${0.1}" /> 	 <!-- chassis_width__mdu +0.01 From front wheel joint to back wheel joint -->
+  <xacro:property name="chassis_height_mdu" value="0.1" /> 				 <!-- From front wheel joint to head rest -->
   <xacro:property name="chassis_weight_mdu" value="${15.0}" />
   <xacro:include filename="$(find mdu_description)/urdf/mdu.gazebo" />
@@ -59,10 +59,14 @@
   <!--link_joint parent='footprint_mdu' child='chassis' xyz="0 0 ${main_wheel_radius_mdu}" rpy="0 0 0" type="fixed"/-->
   <wheel_mdu  lr="rear_left_wheel_mdu" tY="0.02" xyz=" 0 0 0" rpy="${-pi/2} 0 0" wheelWidth="${main_wheel_length_mdu}" wheelRadius="${main_wheel_radius_mdu}" wheelMass="${main_wheel_weight_mdu}" meshFile="wheelchair_wheel"/>
-  <wheel_joint parent="chassis" child ="rear_left_wheel_mdu" xyz="0.05 ${chassis_width_mdu/2 +0.02} 0" rpy="0 0 0" axis="0 1 0"/>
+  <wheel_joint parent="chassis" child ="rear_left_wheel_mdu" xyz="0.0 ${chassis_width_mdu/2 +0.02} 0" rpy="0 0 0" axis="0 1 0"/>
   <wheel_mdu  lr="rear_right_wheel_mdu" tY="0.02" xyz=" 0 0 0" rpy="${pi/2} 0 0" wheelWidth="${main_wheel_length_mdu}" wheelRadius="${main_wheel_radius_mdu}" wheelMass="${main_wheel_weight_mdu}" meshFile="wheelchair_wheel"/>
-  <wheel_joint parent="chassis" child ="rear_right_wheel_mdu" xyz="0.05 ${-chassis_width_mdu/2 - 0.02} 0" rpy="0 0 0" axis="0 1 0"/>
-  <wheel_mdu  lr="front_right_pipe" tY="0.001" xyz=" 0 0 0" rpy="0 ${pi/2} 0" wheelWidth="${0.01}" wheelRadius="${0.015}" wheelMass="${0.5}" meshFile="pipe"/>
-  <!--link_joint parent='front_right_pipe' child='chassis' xyz="${chassis_length_mdu/2 } ${chassis_width__mdu/2 - 0.10} ${(0.082 + 0.00280)}" rpy="0 0 0" type="fixed"/-->
-  <wheel_mdu  lr="front_left_pipe" tY="0.001" xyz=" 0 0 0" rpy="0 ${pi/2} 0" wheelWidth="${0.01}" wheelRadius="${0.015}" wheelMass="${0.5}" meshFile="pipe"/>
-  <link_joint parent='front_left_pipe' child='chassis' xyz="${-chassis_length_mdu/2 } ${-chassis_width__mdu/2 +0.10} ${0.082 + 0.00280}" rpy="0 0 0" type="fixed"/>
+  <wheel_joint parent="chassis" child ="rear_right_wheel_mdu" xyz="0.0 ${-chassis_width_mdu/2 - 0.02} 0" rpy="0 0 0" axis="0 1 0"/>
+  <!--wheel_mdu  lr="front_right_pipe" tY="0.001" xyz=" 0 0 0" rpy="0 ${pi/2} 0" wheelWidth="${0.01}" wheelRadius="${0.005}" wheelMass="${0.5}" meshFile="pipe"/>
+  <wheel_mdu  lr="front_left_pipe" tY="0.001" xyz=" 0 0 0" rpy="0 ${pi/2} 0" wheelWidth="${0.01}" wheelRadius="${0.005}" wheelMass="${0.5}" meshFile="pipe"/-->
+  <!--link_ name="front_left_link" xyz=" 0 0 0" rpy="0 ${3*pi/4} 0" m="${0.1}" length="${0.001}" width="${0.01}" height="${0.01}" />
+  <link_joint parent='chassis' child='front_left_link' xyz="${chassis_length_mdu/2 } ${chassis_width__mdu/2 - 0.01} ${0.082 + 0.00280 - 0.0444}" rpy="0 0 0" type="fixed"/-->
+  <link_ name="front_right_link" xyz=" 0 0 0" rpy="0 0 0" m="${0.1}" length="${0.001}" width="${0.01}" height="${0.01}" />
+  <link_joint parent='chassis' child='front_right_link' xyz="${chassis_length_mdu/2 } ${-chassis_width__mdu/2 + 0.01} ${0.082 + 0.00280 - 0.0444}" rpy="0 0 0" type="fixed"/>
+  <!--link_joint parent='front_right_pipe' child='chassis' xyz="${-chassis_length_mdu/2 } ${chassis_width__mdu/2} ${0.082 + 0.00280 - 0.0444}" rpy="0 0 0" type="fixed"/>
+  <link_joint parent='front_left_pipe' child='chassis' xyz="${-chassis_length_mdu/2 } ${-chassis_width__mdu/2} ${0.082 + 0.00280 - 0.0444}" rpy="0 0 0" type="fixed"/-->
 </robot>

File: src/wheelchair_description/urdf/macros.xacro (robot description, xacro)
@@ -158,3 +158,30 @@
     </joint>
   </xacro:macro>
+  <xacro:macro name="link_" params="name xyz rpy m length width height">
+      <link name="${name}">
+        <collision name='${name}_link_collision'>
+          <geometry>
+            <box size="${length} ${width} ${height}"/>
+          </geometry>
+        </collision>
+        <visual name='${name}_visual'>
+          <origin xyz="${xyz}" rpy="${rpy}" />
+            <geometry>
+              <box size="${length} ${width} ${height}"/>
+          </geometry>
+        </visual>
+        <inertial name="${name}_intertial">
+          <origin xyz="${xyz}" rpy="${rpy}" />
+          <mass value="${m}"/>
+          <box_inertia m="${m}" x="${length}" y="${width}" z ="${height}" />
+        </inertial>
+      </link>
+    </xacro:macro>
+    <xacro:macro name="link_joint" params="parent child xyz rpy type">
+      <joint type="${type}" name="${parent}_${child}_joint">
+        <origin xyz="${xyz}" rpy="${rpy}"/>
+        <parent link="${parent}"/>
+        <child link="${child}"/>
+      </joint>
+    </xacro:macro>
 </robot>

File: src/wheelchair_description/urdf/wheelchair.urdf (robot description, URDF)
Before this commit: robot wheelchair, 22 links, 21 joints
Links:
- removed link front_left_pipe
- removed link front_right_pipe
- added link front_right_link, mass 0.1; collision box size=0.001 0.01 0.01; visual box size=0.001 0.01 0.01
- link chassis: geometry collision box size=0.1 0.15 0.1; collision sphere radius=0.041275
- link person_body: mass 65 -> 1
- link rear_left_leg: geometry collision box size=0.15 0.01 0.01; visual box size=0.15 0.01 0.01
- link rear_left_pipe: geometry collision mesh filename=package://wheelchair_description/meshes/pipe1.stl scale=0.01 0.01 0.01; visual mesh filename=package://wheelchair_description/meshes/pipe1.stl scale=0.01 0.01 0.01
- link rear_left_wheel_mdu: geometry collision cylinder length=0.05 radius=0.08255; visual cylinder length=0.03 radius=0.08255
- link rear_right_leg: geometry collision box size=0.15 0.01 0.01; visual box size=0.15 0.01 0.01
- link rear_right_pipe: geometry collision mesh filename=package://wheelchair_description/meshes/pipe1.stl scale=0.01 0.01 0.01; visual mesh filename=package://wheelchair_description/meshes/pipe1.stl scale=0.01 0.01 0.01
- link rear_right_wheel_mdu: geometry collision cylinder length=0.05 radius=0.08255; visual cylinder length=0.03 radius=0.08255
Joints:
- removed joint base_rear_left_leg_joint
- removed joint base_rear_right_leg_joint
- removed joint front_left_pipe_chassis_joint
- removed joint rear_left_pipe_front_left_pipe_joint
- removed joint rear_right_pipe_front_right_pipe_joint
- added joint axle_rear_left_leg_joint: type fixed, parent axle, child rear_left_leg, origin xyz=0 0.061784 0 rpy=0 -0.785398163397 0
- added joint axle_rear_right_leg_joint: type fixed, parent axle, child rear_right_leg, origin xyz=0 -0.061784 0 rpy=0 -0.785398163397 0
- added joint chassis_front_right_link_joint: type fixed, parent chassis, child front_right_link, origin xyz=0.05 -0.065 0.0404 rpy=0 0 0
- added joint rear_left_pipe_chassis_joint: type fixed, parent rear_left_pipe, child chassis, origin xyz=-0.0132 -0.06 0.11 rpy=0 1.57079632679 0
- added joint rear_right_pipe_front_right_link_joint: type fixed, parent rear_right_pipe, child front_right_link, origin xyz=0 0 0 rpy=0 0 0
- joint chassis_rear_left_wheel_mdu_joint: origin xyz=0.05 0.145 0 rpy=0 0 0 -> xyz=0.0 0.095 0 rpy=0 0 0
- joint chassis_rear_right_wheel_mdu_joint: origin xyz=0.05 -0.145 0 rpy=0 0 0 -> xyz=0.0 -0.095 0 rpy=0 0 0
- joint rear_left_leg_rear_left_pipe_joint: origin xyz=0 0 -0.26 rpy=0 0 0 -> xyz=-0.15 0 0 rpy=0 -0.785398163397 0
- joint rear_right_leg_rear_right_pipe_joint: origin xyz=0 0 -0.26 rpy=0 0 0 -> xyz=-0.15 0 0 rpy=0 -0.785398163397 0

File: src/wheelchair_description/urdf/wheelchair.xacro (robot description, xacro)
@@ -3,5 +3,7 @@
   <xacro:property name="legs_width" value="0.01" />
   <xacro:property name="legs_length" value="0.01" />
+  <xacro:property name="rear_legs_length" value="0.15" />
   <xacro:property name="legs_height" value="0.16" />
+  <xacro:property name="rear_legs_height" value="0.01" />
   <xacro:property name="legs_weight" value="0.25" />
   <xacro:property name="main_wheel_length" value="0.0356884" />
@@ -62,9 +64,11 @@
   <chassis name="front_left_leg" xyz="0 0 ${-legs_height/2}" rpy="0 0 0" m="${legs_weight}" chassisLength="${legs_length}" chassisWidth="${legs_width}" chassisHeight="${legs_height}"/>
   <link_joint parent="base" child ="front_left_leg" xyz="${chair_length} ${chair_width/2} 0" rpy="0 0 0" type="fixed"/>
-   <chassis name="rear_left_leg" xyz="0 0 ${-(legs_height + 0.1)/2}" rpy="0 0 0" m="${legs_weight}" chassisLength="${legs_length}" chassisWidth="${legs_width}" chassisHeight="${legs_height + 0.1}"/>
-  <link_joint parent="base" child ="rear_left_leg" xyz="0 ${chair_width/2 - 0.1} 0" rpy="0 0 0" type="fixed"/>
-<chassis name="rear_right_leg" xyz="0 0 ${-(legs_height + 0.1)/2}" rpy="0 0 0" m="${legs_weight}" chassisLength="${legs_length}" chassisWidth="${legs_width}" chassisHeight="${legs_height +0.1}"/>
-  <link_joint parent="base" child ="rear_right_leg" xyz="0 ${-chair_width/2 + 0.1} 0" rpy="0 0 0" type="fixed"/>
-  <chassis name="front_right_leg" xyz="0 0 ${-legs_height/2}" rpy="0 0 0" m="${legs_weight}" chassisLength="${legs_length}" chassisWidth="${legs_width}" chassisHeight="${legs_height}"/>
+  <link_ name="rear_left_leg" xyz=" ${-rear_legs_length/2} 0 0" rpy="0 0 0" m="${legs_weight}" length="${rear_legs_length}" width="${legs_width}" height="${rear_legs_height}" />
+  <link_ name="rear_right_leg" xyz=" ${-rear_legs_length/2} 0 0" rpy="0 0 0" m="${legs_weight}" length="${rear_legs_length}" width="${legs_width}" height="${rear_legs_height}" />
+   <!--chassis name="rear_left_leg" xyz="0 0 ${rear_legs_length/2}" rpy="0 0 0" m="${legs_weight}" chassisLength="${rear_legs_length}" chassisWidth="${legs_width}" chassisHeight="${rear_legs_height}"/-->
+  <link_joint parent="axle" child ="rear_left_leg" xyz="0 ${chair_width/2 - 0.1} 0" rpy="0 ${-pi/4} 0" type="fixed"/>
+<!--chassis name="rear_right_leg" xyz="-0.05 0 ${-(rear_legs_height + 0.1)/2}" rpy="0 ${pi/4} 0" m="${legs_weight}" chassisLength="${rear_legs_length}" chassisWidth="${legs_width}" chassisHeight="${rear_legs_height}"/-->
+  <link_joint parent="axle" child ="rear_right_leg" xyz="0 ${-chair_width/2 + 0.1} 0" rpy="0 ${-pi/4} 0" type="fixed"/>
+  <chassis name="front_right_leg" xyz="${-legs_height/2} ${-legs_height/2} ${-legs_height/2}" rpy="0 0 0" m="${legs_weight}" chassisLength="${legs_length}" chassisWidth="${legs_width}" chassisHeight="${legs_height}"/>
   <link_joint parent="base" child ="front_right_leg" xyz="${chair_length} ${-chair_width/2} 0" rpy="0 0 0" type="fixed"/>
   <wheel  lr="front_left_leg_rev" tY="0.02" xyz=" 0 0 0" rpy="0 0 0" wheelWidth="${0.1}" wheelRadius="${legs_width}" wheelMass="${legs_weight}" meshFile="wheelchair_wheel_rev"/>
@@ -80,13 +84,15 @@
   <wheel  lr="front_right_wheel" tY="0.001" xyz=" 0 0 0" rpy="${pi/2} 0 0" wheelWidth="${small_wheel_length}" wheelRadius="${small_wheel_radius}" wheelMass="${small_wheel_weight}" meshFile="wheelchair_wheel_small"/>
   <wheel_joint parent="front_right_leg_rev" child ="front_right_wheel" xyz="0.017 0 ${-0.07352}" rpy="0 0 0" axis="0 1 0"/>
-   <sphere_ name="person_body" xyz="0 0 0" rpy="0 0 0" m="65" r="${chair_width/2 -0.02}"/>
+   <sphere_ name="person_body" xyz="0 0 0" rpy="0 0 0" m="1" r="${chair_width/2 -0.02}"/>
    <link_joint parent="base" child ="person_body" xyz="${chair_width/2 -0.02} 0 ${chair_width/2 -0.02}" rpy="0 0 0" type="fixed"/>
    <sphere_ name="person_head" xyz="0 0 0" rpy="0 0 0" m="5" r="${chair_width/4}"/>
    <link_joint parent="person_body" child ="person_head" xyz="0 0 ${chair_width/2}" rpy="0 0 0" type="fixed"/>
-   <wheel  lr="rear_right_pipe" tY="0.001" xyz=" ${-0.025} 0 -0.01" rpy="0 ${pi/2} 0" wheelWidth="${0.05}" wheelRadius="${0.04}" wheelMass="${0.5}" meshFile="pipe"/>
-   <link_joint parent="rear_right_leg" child ="rear_right_pipe" xyz="0 0 ${-legs_height-0.1}" rpy="0 0 0" type="fixed"/>
-   <wheel  lr="rear_left_pipe" tY="0.001" xyz=" ${-0.025} 0 -0.01" rpy="0 ${pi/2} 0" wheelWidth="${0.05}" wheelRadius="${0.04}" wheelMass="${0.5}" meshFile="pipe"/>
-   <link_joint parent="rear_left_leg" child ="rear_left_pipe" xyz="0 0 ${-legs_height-0.1}" rpy="0 0 0" type="fixed"/>
-    <link_joint parent="rear_left_pipe" child ="front_left_pipe" xyz="0 0 0" rpy="0 0 0" type="fixed"/>
-    <link_joint parent="rear_right_pipe" child ="front_right_pipe" xyz="0 0 0" rpy="0 0 0" type="fixed"/>
+   <wheel  lr="rear_right_pipe" tY="0.001" xyz="0 0 ${0.03824}" rpy="0 0 0" wheelWidth="${0.05}" wheelRadius="${0.005}" wheelMass="${0.5}" meshFile="pipe1"/>
+   <wheel  lr="rear_left_pipe" tY="0.001"  xyz="0 0 ${0.03824}" rpy="0 0 0" wheelWidth="${0.05}" wheelRadius="${0.005}" wheelMass="${0.5}" meshFile="pipe1"/>
+   <link_joint parent="rear_right_leg" child ="rear_right_pipe" xyz="${-rear_legs_length} 0 0" rpy="0 ${-pi/4} 0" type="fixed"/>
+   <link_joint parent="rear_left_leg" child ="rear_left_pipe" xyz="${-rear_legs_length} 0 0" rpy="0 ${-pi/4} 0" type="fixed"/>
+    <!--link_joint parent="rear_left_pipe" child ="front_left_pipe" xyz="0 0 0" rpy="0 0 0" type="fixed"/-->
+    <link_joint parent="rear_left_pipe" child ="chassis"  xyz="-0.0132 -0.06 0.11" rpy="0 ${pi/2} 0" type="fixed"/>
+    <link_joint parent="rear_right_pipe" child ="front_right_link" xyz="0 0 0" rpy="0 0 0" type="fixed"/>
+    <!--link_joint parent="rear_left_pipe" child ="front_left_link" xyz="0 0 0" rpy="0 0 0" type="fixed"/-->
 </robot>
